File: ali/v2/thermocouples/microcontroller.kicad_sch (KiCad schematic)
At the start: 41 parts, among them J1 Conn_02x01, J2 Conn_01x05, J3 USB_C_Receptacle_USB2.0_16P, J4 Conn_01x15, J5 Conn_02x09_Counter_Clockwise, J6 Screw_Terminal_01x02, SW1 SKRPANE010, U1 STM32H563RIV6, U2 AP2112K-3.3, Y1 25 MHz

Commit message: mfw tcs
Parts:
- added C12: 22uF, APRL_Passive:C_0805, symbol Device:C_Small
- added C13, C14: 10nF, APRL_Passive:C_0603, symbol Device:C_Small
- added U2: UCC33420-Q1, APRL_Package_QFN:VSON-12_4x5mm_P0.65mm, symbol APRL_Power:UCC33420
- renumbered C12 to C15, C13 to C16, C14 to C17, C15 to C18, C16 to C19, C17 to C20, D3 to D1, D4 to D2, D5 to D3, D1 to D4, D2 to D5, R5 to R3, R3 to R4, R4 to R5, U2 to U3
Connections:
- net +5V: now also C14.2, U2.7 (SEL), U2.8 (VCC); no longer F2.2
- net ADC_RESET: now also J4.6 (Pin_6), U1.55 (PC11); no longer J4.4 (Pin_4), U1.3 (PC14)
- net ADC_START: now also J4.10 (Pin_10); no longer J4.3 (Pin_3)
- net GND: now also C14.1, U2.10 (GNDS), U2.11 (GNDS), U2.12 (GNDS), U2.9 (GNDS); no longer J6.1 (Pin_1)
- net PC10: now also J4.12 (Pin_12); no longer J4.13 (Pin_13)
- net PE0: now also J4.5 (Pin_5); no longer J4.6 (Pin_6)
- net SCLK: now also J4.7 (Pin_7); no longer J4.10 (Pin_10)
- net PB8 renamed I2C4_SCL
- net I2C4_SCL: now also J4.4 (Pin_4); no longer J4.7 (Pin_7)
- net PB9 renamed I2C4_SDA
- net I2C4_SDA: now also J4.3 (Pin_3); no longer J4.5 (Pin_5)
- net PC0 renamed CJC_~{RESET}
- removed net PC11: J4.12 (Pin_12), U1.55 (PC11)
- new net: C12.1, C13.2, F2.2, U2.1 (EN/FLT), U2.2 (VINP)
- new net Earth: C12.2, C13.1, J6.1 (Pin_1), U2.3 (GNDP), U2.4 (GNDP), U2.5 (GNDP), U2.6 (GNDP)
- new net PC14: U1.3 (PC14)
- no-connect marks 18 -> 19
Other:
- note added: "GPIO"
- note added: "POWER"
- note added: "chip has a weird footprint in stock at lcsc btw"
- note added: "fsw is 64.5 MHz (which is kinda crazy) I wasn't able to find a bead thats a good fit so it is what it is"
- note removed: "GPIO Banks"
- moved on the sheet: C1, C10, C11, C15, C16, C17, C18, C19, C2, C20, C3, C4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
