File: ali/v2/thermocouples/thermocouples.kicad_pcb (KiCad board)
At the start: 4 copper layers, 76 x 76 mm, 130 parts, among them J1 Conn_02x01, J10 Conn_01x04_MountingPin, J11 Conn_01x04_MountingPin, J12 Conn_01x04_MountingPin, J13 Conn_01x04_MountingPin, J14 Conn_01x04_MountingPin, J2 Conn_01x05_MountingPin, J3 USB_C_Receptacle_USB2.0_16P, J4 Conn_01x15, J5 Conn_02x09_Counter_Clockwise, J6 Screw_Terminal_01x02, J7 Conn_01x03, J8 Hanrun HY951180A, J9 Conn_01x04_MountingPin, SW1 SKRPANE010, U1 STM32H563RIVx, U2 AP2112K-3.3, U3 TJA1462ATK, U4 LAN8742AI, U5 ADS124S08, Y1 25 MHz, Y2 25 MHz

Commit message: mfw tcs
Parts:
- removed the C29 at (106.2, 128.1)
- removed the C30 at (106.2, 98.9)
- removed the C31 at (108.4, 125.7)
- removed the C36 at (115.8, 85.5)
- removed the C37 at (106.2, 123.3)
- removed the C48 at (114.6, 89.8)
- removed the U3 at (152.8, 104.0)
- added C12: 22uF, APRL_Passive:C_0805, F.Cu at (162.1, 85.0)
- added C13: 10nF, APRL_Passive:C_0603, F.Cu at (164.0, 85.0)
- added C14: 10nF, APRL_Passive:C_0603, F.Cu at (153.5, 79.6)
- added C33: 1nF, APRL_Passive:C_0603, F.Cu at (124.4, 88.1)
- added C34: 10nF, APRL_Passive:C_0603, F.Cu at (126.6, 76.4)
- added C45: 10nF, APRL_Passive:C_0603, F.Cu at (126.6, 104.0)
- added C53: 1nF, APRL_Passive:C_0603, F.Cu at (124.4, 110.9)
- added C54: 1nF, APRL_Passive:C_0603, F.Cu at (124.4, 120.2)
- added C55: 100nF, APRL_Passive:C_0603, B.Cu at (131.1, 103.1)
- added C56: 100nF, APRL_Passive:C_0603, B.Cu at (115.2, 77.4)
- added C57: 100nF, APRL_Passive:C_0603, B.Cu at (115.1, 86.7)
- added C58: 100nF, APRL_Passive:C_0603, B.Cu at (115.1, 95.8)
- added C59: 100nF, APRL_Passive:C_0603, B.Cu at (115.1, 105.1)
- added C60: 100nF, APRL_Passive:C_0603, B.Cu at (115.1, 114.2)
- added C61: 100nF, APRL_Passive:C_0603, B.Cu at (115.1, 123.5)
- added R33: 1k, APRL_Passive:R_0603, F.Cu at (124.4, 103.2)
- added R34: 10M, APRL_Passive:R_0603, F.Cu at (122.2, 93.3)
- added R35: 10M, APRL_Passive:R_0603, F.Cu at (122.2, 102.5)
- added R36: 10M, APRL_Passive:R_0603, F.Cu at (122.2, 115.0)
- added R37: 10M, APRL_Passive:R_0603, F.Cu at (122.2, 124.3)
- added R38: 1k, APRL_Passive:R_0603, F.Cu at (124.4, 114.1)
- added R39: 1k, APRL_Passive:R_0603, F.Cu at (124.4, 123.4)
- added R40: 1k, APRL_Passive:R_0603, F.Cu at (124.4, 112.5)
- added R41: 1k, APRL_Passive:R_0603, F.Cu at (124.4, 121.8)
- added R42: 10M, APRL_Passive:R_0603, F.Cu at (122.2, 111.8)
- added R43: 10M, APRL_Passive:R_0603, F.Cu at (122.2, 121.1)
- added R44: 4.7k, APRL_Passive:R_0603, B.Cu at (138.3, 93.7)
- added R45: 4.7k, APRL_Passive:R_0603, B.Cu at (140.0, 92.2)
- added R46: 4.7k, APRL_Passive:R_0603, B.Cu at (122.2, 101.9)
- added R47: 4.7k, APRL_Passive:R_0603, B.Cu at (132.7, 95.7)
- added R48: 4.7k, APRL_Passive:R_0603, B.Cu at (122.2, 100.3)
- added R49: 4.7k, APRL_Passive:R_0603, B.Cu at (129.7, 92.3)
- added R50: 4.7k, APRL_Passive:R_0603, B.Cu at (128.0, 91.4)
- added R51: 4.7k, APRL_Passive:R_0603, B.Cu at (117.1, 109.1)
- added R52: 4.7k, APRL_Passive:R_0603, B.Cu at (116.3, 107.5)
- added U10: TMP117AIDRVR, Package_SON:WSON-6-1EP_2x2mm_P0.65mm_EP1x1.6mm, F.Cu at (113.9, 121.5)
- added U11: TMP117AIDRVR, Package_SON:WSON-6-1EP_2x2mm_P0.65mm_EP1x1.6mm, F.Cu at (114.0, 75.4)
- added U12: TMP117AIDRVR, Package_SON:WSON-6-1EP_2x2mm_P0.65mm_EP1x1.6mm, F.Cu at (113.9, 112.2)
- added U13: TMP117AIDRVR, Package_SON:WSON-6-1EP_2x2mm_P0.65mm_EP1x1.6mm, F.Cu at (113.9, 93.8)
- added U2: UCC33420-Q1, APRL_Package_QFN:VSON-12_4x5mm_P0.65mm, F.Cu at (157.6, 84.7)
- added U5: LAN8742AI, APRL_Package_QFN:VQFN-24-1EP_4x4mm_P0.5mm_EP2.5x2.5mm_ThermalVias, F.Cu at (146.3, 121.7)
- added U7: TCA9543A, Package_SO:Texas_HTSSOP-14-1EP_4.4x5mm_P0.65mm_EP3.4x5mm_Mask3.155x3.255mm_ThermalVias, B.Cu at (127.9, 99.4)
- added U8: TMP117AIDRVR, Package_SON:WSON-6-1EP_2x2mm_P0.65mm_EP1x1.6mm, F.Cu at (113.9, 103.1)
- added U9: TMP117AIDRVR, Package_SON:WSON-6-1EP_2x2mm_P0.65mm_EP1x1.6mm, F.Cu at (113.9, 84.7)
- C30: renamed from C27; value 10pF -> 15pF
- C31: renamed from C28; value 10pF -> 15pF
- C32, C41, C42, C49, C50: value 10nF -> 1nF
- C35: value 100nF -> 10nF; moved to F.Cu
- C38: value 1nF -> 100nF; moved to B.Cu
- C39: value 1nF -> 22uF; footprint APRL_Passive:C_0603 -> APRL_Passive:C_0805; moved to B.Cu
- C44, C51, C52: value 1nF -> 10nF
- C8, C9: value 10pF -> 15pF
- D10, D12, D14, D16, D6, D8: value SMF5V0A -> SMF7V0A
- J10, J11, J12, J13, J14, J9: value Conn_01x04_MountingPin -> Conn_01x02; footprint APRL_Connector_Molex:Molex_CLIK-Mate_503159-0401_1x04-1MP_P1.50mm_Vertical -> APRL_Connector:PCC-SMP-V-K
- J2: value Conn_01x05_MountingPin -> Conn_01x05
- J8: value Hanrun HY951180A -> Vertical Ethernet
- R19, R20, R26, R27, R28, R29: value 1k -> 10M
- R21: value 10R -> 1k; moved to F.Cu
- R23: value 1k -> 10R; moved to B.Cu
- R24: value 100k -> 1k
- U1: value STM32H563RIVx -> STM32H563RIV6
- U4: value LAN8742AI -> TJA1462ATK; footprint Package_DFN_QFN:VQFN-24-1EP_4x4mm_P0.5mm_EP2.5x2.5mm_ThermalVias -> APRL_Package_QFN:HVSON-8-1EP_3x3mm_P0.65mm_EP1.6x2.4mm_ThermalVias
- moved D6 52.1 mm to (117.6, 75.2), turned to 180 degrees
- moved C52 52.1 mm to (126.6, 122.6), turned to -90 degrees
- moved J9 51.2 mm to (119.0, 78.9), turned to -90 degrees
- moved R19 50.9 mm to (122.2, 78.1), turned to 90 degrees
- moved C50 50.5 mm to (124.4, 125.0), turned to 180 degrees
- moved D7 50.0 mm to (112.8, 74.1), turned to 90 degrees
- moved J14 48.3 mm to (119.0, 124.9), turned to -90 degrees
- moved D17 45.2 mm to (112.8, 120.0), turned to 90 degrees
- moved D16 44.7 mm to (117.6, 121.3), turned to 180 degrees
- moved C39 43.7 mm to (128.5, 80.7)
- moved R22 42.4 mm to (124.4, 86.5)
- moved R25 36.6 mm to (124.4, 84.9)
- moved C41 36.3 mm to (124.4, 83.3), turned to 0 degrees
- moved R27 34.7 mm to (122.2, 84.2), turned to 90 degrees
- moved U4 30.2 mm to (161.8, 104.0), turned to 0 degrees
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- renumbered C12 to C15, C13 to C16, C14 to C17, C15 to C18, C16 to C19, C17 to C20, C18 to C21, C19 to C22, C20 to C23, C21 to C24, C22 to C25, C23 to C26, C24 to C27, C25 to C28, C26 to C29, C33 to C36, C34 to C37, C45 to C48, D3 to D1, D4 to D2, D5 to D3, D1 to D4, D2 to D5, R5 to R3, R3 to R4, R4 to R5, U2 to U3, U5 to U6
Connections:
- net /Microcontroller/PC0 renamed /CJC Sensors/~{RESET}
- C26 pad 1: Net-(U4-VDDCR) -> Net-(U5-VDDCR)
- C27 pad 1: Net-(U4-VDDCR) -> Net-(U5-VDDCR)
- C30 pad 1: Net-(U4-XTAL1/CLKIN) -> Net-(U5-XTAL1/CLKIN)
- C31 pad 1: Net-(U4-XTAL2) -> Net-(U5-XTAL2)
- C32 pad 1: /ADC/AIN7 -> /ADC/AIN10
- C32 pad 2: /ADC/AIN6 -> GND
- C35 pad 1: Net-(U5-AVDD) -> /ADC/AIN9
- C35 pad 2: GND -> /ADC/AIN8
- C38 pad 1: GND -> Net-(U6-AVDD)
- C38 pad 2: /ADC/AIN7 -> GND
- C39 pad 1: /ADC/AIN2 -> Net-(U6-AVDD)
- C40 pad 1: /ADC/AIN8 -> GND
- C40 pad 2: GND -> /ADC/AIN11
- C41 pad 1: /ADC/AIN3 -> GND
- C41 pad 2: /ADC/AIN2 -> /ADC/AIN9
- C42 pad 1: /ADC/AIN9 -> /ADC/AIN6
- C42 pad 2: /ADC/AIN8 -> GND
- C43 pad 1: GND -> /ADC/AIN4
- C43 pad 2: /ADC/AIN3 -> GND
- C44 pad 1: GND -> /ADC/AIN7
- C44 pad 2: /ADC/AIN9 -> /ADC/AIN6
- C46 pad 1: /ADC/AIN4 -> GND
- C46 pad 2: GND -> /ADC/AIN7
- C47 pad 1: /ADC/AIN10 -> GND
- C47 pad 2: GND -> /ADC/AIN5
- C49 pad 1: /ADC/AIN5 -> /ADC/AIN2
- C49 pad 2: /ADC/AIN4 -> GND
- C50 pad 1: /ADC/AIN11 -> /ADC/AIN0
- C50 pad 2: /ADC/AIN10 -> GND
- C51 pad 1: GND -> /ADC/AIN3
- C51 pad 2: /ADC/AIN5 -> /ADC/AIN2
- C52 pad 1: GND -> /ADC/AIN1
- C52 pad 2: /ADC/AIN11 -> /ADC/AIN0
- F2 pad 2: +5V -> Net-(U2-EN/FLT)
- J10 pad 1: +5V -> Net-(D8-A1)
- J10 pad 2: Net-(D8-A1) -> Net-(D9-A1)
- J11 pad 1: +5V -> Net-(D10-A1)
- J11 pad 2: Net-(D10-A1) -> Net-(D11-A1)
- J12 pad 1: +5V -> Net-(D12-A1)
- J12 pad 2: Net-(D12-A1) -> Net-(D13-A1)
- J13 pad 1: +5V -> Net-(D14-A1)
- J13 pad 2: Net-(D14-A1) -> Net-(D15-A1)
- J14 pad 1: +5V -> Net-(D16-A1)
- J14 pad 2: Net-(D16-A1) -> Net-(D17-A1)
- J4 pad 10: /ADC/SCLK -> /ADC/START
- J4 pad 12: /Microcontroller/PC11 -> /Microcontroller/PC10
- J4 pad 13: /Microcontroller/PC10 -> unconnected-(J4-Pin_13-Pad13)
- J4 pad 3: /ADC/START -> /CJC Sensors/SDA
- J4 pad 4: /ADC/RESET -> /CJC Sensors/SCL
- J4 pad 5: /Microcontroller/PB9 -> /Microcontroller/PE0
- J4 pad 6: /Microcontroller/PE0 -> /ADC/RESET
- J4 pad 7: /Microcontroller/PB8 -> /ADC/SCLK
- J6 pad 1: GND -> Earth
- J9 pad 1: +5V -> Net-(D6-A1)
- J9 pad 2: Net-(D6-A1) -> Net-(D7-A1)
- R14 pad 2: Net-(U4-RXER/PHYAD0) -> Net-(U5-RXER/PHYAD0)
- R15 pad 1: Net-(U4-RBIAS) -> Net-(U5-RBIAS)
- R19 pad 1: Net-(D6-A1) -> +5V
- R19 pad 2: /ADC/AIN0 -> Net-(D6-A1)
- R20 pad 1: Net-(D8-A1) -> +5V
- R20 pad 2: /ADC/AIN6 -> Net-(D8-A1)
- R21 pad 1: Net-(U5-AVDD) -> Net-(D6-A1)
- R21 pad 2: +5V -> /ADC/AIN10
- R22 pad 1: Net-(D7-A1) -> Net-(D8-A1)
- R22 pad 2: /ADC/AIN1 -> /ADC/AIN8
- R23 pad 1: Net-(D9-A1) -> Net-(U6-AVDD)
- R23 pad 2: /ADC/AIN7 -> +5V
- R24 pad 1: +5V -> Net-(D7-A1)
- R24 pad 2: Net-(U5-AINCOM) -> /ADC/AIN11
- R25 pad 1: Net-(D10-A1) -> Net-(D9-A1)
- R25 pad 2: /ADC/AIN2 -> /ADC/AIN9
- R26 pad 1: Net-(D12-A1) -> Net-(D7-A1)
- R26 pad 2: /ADC/AIN8 -> GND
- R27 pad 1: Net-(D11-A1) -> Net-(D9-A1)
- R27 pad 2: /ADC/AIN3 -> GND
- R28 pad 1: Net-(D13-A1) -> +5V
- R28 pad 2: /ADC/AIN9 -> Net-(D10-A1)
- R29 pad 1: Net-(D14-A1) -> +5V
- R29 pad 2: /ADC/AIN4 -> Net-(D12-A1)
- R30 pad 1: Net-(D16-A1) -> Net-(D10-A1)
- R30 pad 2: /ADC/AIN10 -> /ADC/AIN6
- R31 pad 1: Net-(D15-A1) -> Net-(D12-A1)
- R31 pad 2: /ADC/AIN5 -> /ADC/AIN4
- R32 pad 1: Net-(D17-A1) -> Net-(D11-A1)
- R32 pad 2: /ADC/AIN11 -> /ADC/AIN7
- U1 pad 3: /ADC/RESET -> /Microcontroller/PC14
- U1 pad 55: /Microcontroller/PC11 -> /ADC/RESET
- U1 pad 63: /Microcontroller/PB8 -> /CJC Sensors/SCL
- U1 pad 64: /Microcontroller/PB9 -> /CJC Sensors/SDA
- U4 pad 1: +3.3V -> /Connectivity/FDCAN_TX
- U4 pad 2: /Connectivity/LED2-INTSEL -> GND
- U4 pad 3: /Connectivity/LED1-REGOFF -> +5V
- U4 pad 4: Net-(U4-XTAL2) -> /Connectivity/FDCAN_RX
- U4 pad 5: Net-(U4-XTAL1/CLKIN) -> +3.3V
- U4 pad 6: Net-(U4-VDDCR) -> Net-(J7-Pin_2)
- U4 pad 7: /Connectivity/ETH_RXD1 -> Net-(J7-Pin_1)
- U4 pad 8: /Connectivity/ETH_RXD0 -> /Connectivity/FDCAN_STDBY
- U4 pad 9: +3.3V -> GND
- U6 pad 1: Net-(U5-AINCOM) -> GND
- U6 pad 17: unconnected-(U5-CLK-Pad17) -> GND
- U6 pad 26: Net-(U5-AVDD) -> Net-(U6-AVDD)
- U6 pad 29: GND -> unconnected-(U6-REFN0-Pad29)
- U6 pad 30: +5V -> unconnected-(U6-REFP0-Pad30)
- Y2 pad 1: Net-(U4-XTAL1/CLKIN) -> Net-(U5-XTAL1/CLKIN)
- Y2 pad 3: Net-(U4-XTAL2) -> Net-(U5-XTAL2)
Routing:
- net +5V: track 6.99 -> 144.5 mm, vias 12 -> 11
- net +3.3V: track 5.28 -> 107.9 mm, vias 34 -> 38
- net Net-(U11-SDA): track 0.00 -> 56.4 mm, vias 0 -> 3
- net Net-(U11-SCL): track 0.00 -> 54.4 mm, vias 0 -> 3
- net /CJC Sensors/SCL: track 0.00 -> 47.3 mm, vias 0 -> 1
- net /CJC Sensors/SDA: track 0.00 -> 45.0 mm, vias 0 -> 3
- net Net-(U10-SDA): track 0.00 -> 42.6 mm, vias 0 -> 3
- net /CJC Sensors/~{RESET}: track 42.0 -> 80.2 mm, vias 0 -> 2
- net Net-(U10-SCL): track 0.00 -> 37.1 mm, vias 0 -> 3
- net /Microcontroller/PB9: track 26.2 -> 0.00 mm, vias 1 -> 0
- net /Microcontroller/PB8: track 24.9 -> 0.00 mm, vias 1 -> 0
- net /Microcontroller/PC11: track 24.9 -> 0.00 mm, vias 1 -> 0
- net Net-(U5-XTAL1/CLKIN): track 0.00 -> 15.1 mm
- net Net-(U4-XTAL1/CLKIN): track 15.1 -> 0.00 mm
- net Net-(D13-A1): track 4.46 -> 15.7 mm
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- added copper zone on F.Cu, net Earth
- added copper zone on F.Cu, net Net-(U2-EN/FLT)
- added copper zone on F.Cu, net Net-(U5-VDDCR)
- added copper zone on B.Cu, net Net-(U6-AVDD)
- added copper zone on F.Cu, net Net-(U6-AVDD)
- removed copper zone on F.Cu, net Net-(U4-VDDCR)
- removed copper zone on B.Cu, net Net-(U5-AVDD)
- removed copper zone on F.Cu, net Net-(U5-AVDD)
Other:
- board size 76 x 76 mm -> 85 x 76 mm
- board text added: "DAQ"
- board text added: "THERMOCOUPLE"
- board text added: "USB PWR"
- board text removed: "L1"
- board text removed: "L2"
- board text removed: "L3"
- board text removed: "L4"
- board text removed: "L5"
- board text removed: "L6"
- board text removed: "THERMOCOUPLE DAQ"
- board text removed: "USB POWER"

Commit message: mfw pts
Parts:
- moved R50 1.87 mm to (126.2, 90.9)
- moved R49 0.71 mm to (129.2, 91.8)
Connections:
- J4 pad 13: unconnected-(J4-Pin_13-Pad13) -> /Microcontroller/PA15
- J4 pad 14: /Microcontroller/PA15 -> /Microcontroller/PA9
- U1 pad 45: unconnected-(U1-PA9-Pad45) -> /Microcontroller/PA9
Routing:
- net /Microcontroller/PA9: track 0.00 -> 39.3 mm, vias 0 -> 2
- net /Microcontroller/PA15: track 33.9 -> 30.2 mm
- net GND: vias 305 -> 353

Commit message: Swap to sync'd ADS1261s on LC, update README and clean up Just scripts, some frame changes too.
Other:
- board text added: "REV ${REV}"
- board text removed: "REV 1A"

Commit message: Minor thermocouple updates
Parts:
- removed J4: Conn_01x15, APRL_Connector_Molex:Molex_CLIK-Mate_503159-1501_1x15-1MP_P1.50mm_Vertical
- added J15: Conn_01x15, APRL_Connector_Molex:Molex_CLIK-Mate_503159-1501_1x15-1MP_P1.50mm_Vertical, F.Cu at (131.9, 73.2)
- added R53: 10k, APRL_Passive:R_0603, F.Cu at (157.5, 104.8)
- added R54: 10k, APRL_Passive:R_0603, F.Cu at (157.5, 107.6)
- moved D1 7.00 mm to (164.9, 110.6)
- moved D2 7.00 mm to (164.9, 108.8)
- moved D3 7.00 mm to (164.9, 107.0)
- moved R3 7.00 mm to (161.7, 110.6)
- moved R6 7.00 mm to (161.7, 108.8)
- moved R7 7.00 mm to (161.7, 107.0)
- moved R5 3.75 mm to (152.9, 87.1), turned to 0 degrees
- moved D5 2.05 mm to (152.9, 88.7), turned to 0 degrees
- moved C14 1.51 mm to (155.0, 79.8)
- moved C15 1.51 mm to (153.2, 79.9)
- moved C16 1.51 mm to (151.2, 79.9)
- moved C17 1.51 mm to (149.2, 79.9)
- moved C18 1.51 mm to (153.2, 83.8)
- moved C19 1.51 mm to (151.2, 83.8)
- moved C20 1.51 mm to (149.2, 83.8)
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- renumbered J13 to J10, J12 to J11, J11 to J12, J10 to J13, J9 to J14, J14 to J9
Connections:
- net Earth renamed GNDPWR
- J5 pad 11: /Microcontroller/PC3 -> /Microcontroller/PB0
- J5 pad 13: /Microcontroller/PC2 -> /Microcontroller/PA4
- J5 pad 15: /CJC Sensors/~{RESET} -> /Microcontroller/PC3
- J5 pad 17: /Microcontroller/PB10 -> /Microcontroller/PC2
- J5 pad 3: /Microcontroller/PA6 -> /Microcontroller/PB13
- J5 pad 5: /Microcontroller/PA5 -> /Microcontroller/PB2
- J5 pad 7: /Microcontroller/PA4 -> /Microcontroller/TIM2_CH4
- J5 pad 9: /Microcontroller/PA3 -> /Microcontroller/PA6
- U1 pad 17: /Microcontroller/PA3 -> /Microcontroller/TIM2_CH4
- U1 pad 2: unconnected-(U1-PC13-Pad2) -> /ADC/CS
- U1 pad 21: /Microcontroller/PA5 -> /ADC/SCLK
- U1 pad 26: /Microcontroller/USER_LED_1 -> /Microcontroller/PB0
- U1 pad 27: /Microcontroller/USER_LED_2 -> /Microcontroller/+5V_SENSE
- U1 pad 28: /Microcontroller/USER_LED_3 -> /Microcontroller/PB2
- U1 pad 29: /Microcontroller/PB10 -> /Microcontroller/TIM2_CH3
- U1 pad 3: /Microcontroller/PC14 -> /ADC/START
- U1 pad 35: unconnected-(U1-PB13-Pad35) -> /Microcontroller/PB13
- U1 pad 36: unconnected-(U1-PB14-Pad36) -> /Microcontroller/USER_LED_1
- U1 pad 39: unconnected-(U1-PD12-Pad39) -> /Microcontroller/USER_LED_2
- U1 pad 40: unconnected-(U1-PC6-Pad40) -> /Microcontroller/USER_LED_3
- U1 pad 43: unconnected-(U1-PC9-Pad43) -> /Microcontroller/PC9
- U1 pad 45: /Microcontroller/PA9 -> unconnected-(U1-PA9-Pad45)
- U1 pad 53: /Microcontroller/PA15 -> /Microcontroller/TIM2_CH1
- U1 pad 54: /Microcontroller/PC10 -> unconnected-(U1-PC10-Pad54)
- U1 pad 55: /ADC/RESET -> unconnected-(U1-PC11-Pad55)
- U1 pad 56: /ADC/DRDY -> /ADC/RESET
- U1 pad 57: /ADC/SCLK -> /ADC/DRDY
- U1 pad 60: /ADC/CS -> /CJC Sensors/SCL
- U1 pad 61: /ADC/START -> /CJC Sensors/SDA
- U1 pad 63: /CJC Sensors/SCL -> /Microcontroller/UART4_RX
- U1 pad 64: /CJC Sensors/SDA -> /Microcontroller/UART4_TX
- U1 pad 65: /Microcontroller/PE0 -> unconnected-(U1-PE0-Pad65)
Routing:
- net /Microcontroller/TIM2_CH3: track 0.00 -> 61.5 mm, vias 0 -> 4
- net /Microcontroller/PB10: track 53.2 -> 0.00 mm, vias 3 -> 0
- net /ADC/SCLK: track 29.8 -> 80.4 mm, vias 2 -> 5
- net /Microcontroller/PB13: track 0.00 -> 44.7 mm, vias 0 -> 2
- net /Microcontroller/PB2: track 0.00 -> 42.0 mm, vias 0 -> 2
- net /Microcontroller/PB0: track 0.00 -> 41.2 mm, vias 0 -> 2
- net /Microcontroller/PA5: track 40.8 -> 0.00 mm, vias 2 -> 0
- net /Microcontroller/PA9: track 39.3 -> 0.00 mm, vias 2 -> 0
- net /Microcontroller/PA3: track 38.1 -> 0.00 mm, vias 2 -> 0
- net /Microcontroller/PC9: track 0.00 -> 37.7 mm, vias 0 -> 4
- net /Microcontroller/TIM2_CH4: track 0.00 -> 37.5 mm, vias 0 -> 2
- net /Microcontroller/TIM2_CH1: track 0.00 -> 34.5 mm, vias 0 -> 2
- net /Microcontroller/PC10: track 31.4 -> 0.00 mm
- net /Microcontroller/PA15: track 30.2 -> 0.00 mm
- net /Microcontroller/PE0: track 26.5 -> 0.00 mm, vias 1 -> 0
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Other:
- board text removed: "PB0"
- board text removed: "PB1"
- board text removed: "PB2"
