File: ali/v2/thermocouples/connectivity.kicad_sch (KiCad schematic)
At the start: 27 parts, among them J7 Conn_01x03, J8 Vertical Ethernet, U3 TJA1462ATK, U4 LAN8742AI, Y2 25 MHz

Commit message: mfw tcs
Parts:
- J8: LCSC (none) -> C34677
- U4: renamed from U3; footprint Package_SON:HVSON-8-1EP_3x3mm_P0.65mm_EP1.6x2.4mm -> APRL_Package_QFN:HVSON-8-1EP_3x3mm_P0.65mm_EP1.6x2.4mm_ThermalVias
- U5: renamed from U4; footprint Package_DFN_QFN:VQFN-24-1EP_4x4mm_P0.5mm_EP2.5x2.5mm_ThermalVias -> APRL_Package_QFN:VQFN-24-1EP_4x4mm_P0.5mm_EP2.5x2.5mm_ThermalVias
- renumbered C18 to C21, C19 to C22, C20 to C23, C21 to C24, C22 to C25, C23 to C26, C24 to C27, C25 to C28, C26 to C29, C27 to C30, C28 to C31

Commit message: Globally remove LCSC labels, update MPNs and IOCs, add +5V monitoring to DAQs, fix some footprints
Parts:
- C27: MPN GRM21A5C2J471FWA1 -> GRM1885C1H471JA01
- C29: MPN GRM21AR72A224KAC5 -> GRM188R71H224KAC4
- J8: LCSC C34677 -> (none)
- renumbered R8 to R10, R9 to R11, R10 to R12, R11 to R13, R12 to R14, R13 to R15, R14 to R16, R15 to R17, R16 to R18, R17 to R19, R18 to R20

Commit message: Fix 50R/60R widths
Connections:
- net CAN+: now reaches J7.1 (Pin_1), R10.2, U4.7 (CANH)
- net CAN-: now reaches J7.2 (Pin_2), R10.1, U4.6 (CANL)
Changed lines of the file:
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@@
+		)
+	)
+	(label "CAN-"
+		(at 205.7332 67.31 0)
+		(effects
+			(font
+				(size 1.27 1.27)
+			)
+			(justify left bottom)
+		)
+	)
+	(label "CAN+"
+		(at 205.74 62.23 0)
+		(effects
+			(font
+				(size 1.27 1.27)
+			)
+			(justify left bottom)
 		)
 	)

Commit message: Document setup, update template, and use an ampersand when referring to APRL
Other:
- note added: "Isolation is completely defeated if we use CAN"
- note added: "The isolation on this board can only occur if we use an unshielded ethernet cable. For this reason, I think that connecting pins 13 and 14 to GND through a large isolation capacitor and bleed resistor might be a better choice."
Changed lines of the file:
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@@
+		)
+	)
+	(text "The isolation on this board can only occur if we use an unshielded ethernet cable.\nFor this reason, I think that connecting pins 13 and 14 to GND through a large\nisolation capacitor and bleed resistor might be a better choice."
+		(exclude_from_sim no)
+		(at 204.47 156.21 0)
+		(effects
+			(font
+				(size 1.27 1.27)
+			)
 		)
 	)
@@
 		)
 	)
+	(text "Isolation is completely defeated if we use CAN"
+		(exclude_from_sim no)
+		(at 230.632 50.038 0)
+		(effects
+			(font
+				(size 1.27 1.27)
+			)
+		)
+	)
 	(junction
 		(at 100.33 74.93)
@@
 			(width 0)
 			(type default)
+		)
+	)
+	(label "TX+"
+		(at 144.78 74.93 180)
+		(effects
+			(font
+				(size 1.27 1.27)
+			)
+			(justify right bottom)
+		)
+	)
+	(label "LED2-INTSEL"
+		(at 223.52 124.46 180)
+		(effects
+			(font
+				(size 1.27 1.27)
+			)
+			(justify right bottom)
+		)
+	)
+	(label "LED2-INTSEL"
+		(at 111.76 97.79 180)
+		(effects
+			(font
+				(size 1.27 1.27)
+			)
+			(justify right bottom)
+		)
+	)
+	(label "TX-"
+		(at 161.29 119.38 0)
+		(effects
+			(font
+				(size 1.27 1.27)
+			)
+			(justify left bottom)
+		)
+	)
+	(label "RX+"
+		(at 161.29 121.92 0)
+		(effects
+			(font
+				(size 1.27 1.27)
+			)
+			(justify left bottom)
+		)
+	)
+	(label "RX+"
+		(at 144.78 80.01 180)
+		(effects
+			(font
+				(size 1.27 1.27)
+			)
+			(justify right bottom)
+		)
+	)
+	(label "LED1-REGOFF"
+		(at 224.79 114.3 180)
+		(effects
+			(font
+				(size 1.27 1.27)
+			)
+			(justify right bottom)
+		)
+	)
+	(label "LED1-REGOFF"
+		(at 111.76 95.25 180)
+		(effects
+			(font
+				(size 1.27 1.27)
+			)
+			(justify right bottom)
+		)
+	)
+	(label "RX-"
+		(at 144.78 82.55 180)
+		(effects
+			(font
+				(size 1.27 1.27)
+			)
+			(justify right bottom)
+		)
+	)
+	(label "TX+"
+		(at 161.29 114.3 0)
+		(effects
+			(font
+				(size 1.27 1.27)
+			)
+			(justify left bottom)
+		)
+	)
+	(label "TX-"
+		(at 144.78 77.47 180)
+		(effects
+			(font
+				(size 1.27 1.27)
+			)
+			(justify right bottom)
 		)
 	)
@@
 		)
 	)
+	(label "RX-"
+		(at 161.29 127 0)
+		(effects
+			(font
+				(size 1.27 1.27)
+			)
+			(justify left bottom)
+		)
+	)
 	(label "CAN+"
 		(at 205.74 62.23 0)
 		(effects
 			(font
-				(size 1.27 1.27)
-			)
-			(justify left bottom)
-		)
-	)
-	(label "TX+"
-		(at 144.78 74.93 180)
-		(effects
-			(font
-				(size 1.27 1.27)
-			)
-			(justify right bottom)
-		)
-	)
-	(label "LED2-INTSEL"
-		(at 223.52 124.46 180)
-		(effects
-			(font
-				(size 1.27 1.27)
-			)
-			(justify right bottom)
-		)
-	)
-	(label "LED2-INTSEL"
-		(at 111.76 97.79 180)
-		(effects
-			(font
-				(size 1.27 1.27)
-			)
-			(justify right bottom)
-		)
-	)
-	(label "TX-"
-		(at 161.29 119.38 0)
-		(effects
-			(font
-				(size 1.27 1.27)
-			)
-			(justify left bottom)
-		)
-	)
-	(label "RX+"
-		(at 161.29 121.92 0)
-		(effects
-			(font
-				(size 1.27 1.27)
-			)
-			(justify left bottom)
-		)
-	)
-	(label "RX+"
-		(at 144.78 80.01 180)
-		(effects
-			(font
-				(size 1.27 1.27)
-			)
-			(justify right bottom)
-		)
-	)
-	(label "LED1-REGOFF"
-		(at 224.79 114.3 180)
-		(effects
-			(font
-				(size 1.27 1.27)
-			)
-			(justify right bottom)
-		)
-	)
-	(label "LED1-REGOFF"
-		(at 111.76 95.25 180)
-		(effects
-			(font
-				(size 1.27 1.27)
-			)
-			(justify right bottom)
-		)
-	)
-	(label "RX-"
-		(at 144.78 82.55 180)
-		(effects
-			(font
-				(size 1.27 1.27)
-			)
-			(justify right bottom)
-		)
-	)
-	(label "TX+"
-		(at 161.29 114.3 0)
-		(effects
-			(font
-				(size 1.27 1.27)
-			)
-			(justify left bottom)
-		)
-	)
-	(label "TX-"
-		(at 144.78 77.47 180)
-		(effects
-			(font
-				(size 1.27 1.27)
-			)
-			(justify right bottom)
-		)
-	)
-	(label "RX-"
-		(at 161.29 127 0)
-		(effects
-			(font

Commit message: Begin prep for second board review
Parts:
- removed J7: Conn_01x03, APRL_Connector_Molex:Molex_CLIK-Mate_503159-0301_1x03-1MP_P1.50mm_Vertical, symbol Connector_Generic:Conn_01x03
- removed J8: Vertical Ethernet, APRL_Connector:RJ45_Hanrun_HY951180A_Vertical, symbol APRL_Connector:RJ45_Hanrun_HY951180A
- removed R10: 120R, APRL_Passive:R_0603, symbol Device:R_Small_US
- removed R19, R20: 330R, APRL_Passive:R_0603, symbol Device:R_Small_US
- removed U5: LAN8742AI, APRL_Package_QFN:VQFN-24-1EP_4x4mm_P0.5mm_EP2.5x2.5mm_ThermalVias, symbol APRL_Comms:LAN8742A
- added J26: Vertical Ethernet, APRL_Connector:RJ45_Hanrun_HY951180A_Vertical, symbol APRL_Connector:RJ45_Hanrun_HY951180A
- added J8: Conn_01x03, APRL_Connector_Molex:Molex_CLIK-Mate_503159-0301_1x03-1MP_P1.50mm_Vertical, symbol Connector_Generic:Conn_01x03
- added R51: 10k, APRL_Passive:R_0603, symbol Device:R_Small_US
- added R52, R53: 330R, APRL_Passive:R_0603, symbol Device:R_Small_US
- added U7: LAN8742AI, APRL_Package_QFN:VQFN-24-1EP_4x4mm_P0.5mm_EP2.5x2.5mm_ThermalVias, symbol APRL_Comms:LAN8742A
- C25: value 100nF -> 1uF; MPN GRM188R72A104KA35 -> GRM188D72A105KE01
- C26: value 1uF -> 470pF; MPN GRM188D72A105KE01 -> GRM1885C1H471JA01
- C27: value 470pF -> 15pF; MPN GRM1885C1H471JA01 -> GRM1885C2E150FW07
- C28: value 100nF -> 15pF; MPN GRM188R72A104KA35 -> GRM1885C2E150FW07
- C29: value 220nF -> 100nF; MPN GRM188R71H224KAC4 -> GRM188R72A104KA35
- C30: value 15pF -> 220nF; MPN GRM1885C2E150FW07 -> GRM188R71H224KAC4
- C31: value 15pF -> 100nF; MPN GRM1885C2E150FW07 -> GRM188R72A104KA35
- R11: value 1.5k -> 120R; MPN RC0603FR-071K5L -> AC0603FR-07120RL
- R12: value 47R -> 1.5k; MPN RC0603FR-0747RL -> RC0603FR-071K5L
- R16: value 10k -> 47R; MPN RC0603FR-0710KL -> RC0603FR-0747RL
- R17: value 12.1k -> 10k; MPN RT0603BRD0712K1L -> RC0603FR-0710KL
- R18: value 10k -> 12.1k; MPN RC0603FR-0710KL -> RT0603BRD0712K1L
Connections:
- net TX+ is gone; now on net ETH_MDIO: R12.2
- net +3.3V: now also C30.1, R16.1, J26.3 (TCT), J26.5 (RCT), U7.1 (VDD2A), U7.19 (VDD1A), U7.9 (VDDIO); no longer C28.1, R11.1
- net +5V: now also C31.1; no longer C25.1
- net ETH_CRS_DV: now also U7.11 (CRS_DV/MODE2)
- net ETH_MDC: now also U7.13 (MDC)
- net ETH_MDIO: now also U7.12 (MDIO); no longer R11.2
- net ETH_REF_CLK: now also U7.14 (~{INT}/REFCLKO)
- net ETH_RXD0: now also U7.8 (RXD0/MODE0)
- net ETH_RXD1: now also U7.7 (RXD1/MODE1)
- net ETH_TXD0: now also U7.17 (TXD0)
- net ETH_TXD1: now also U7.18 (TXD1)
- net ETH_TX_EN: now also U7.16 (TXEN)
- net ETH_~{RST}: now also U7.15 (~{RST})
- net GND: now also R17.1, J26.13, J26.14, J26.8, J8.3 (Pin_3), R51.2, R52.2, R53.2, U7.25 (VSS); no longer R16.1, R17.2
- net at Y2.1: now also C27.1, U7.5 (XTAL1/CLKIN); no longer C30.1
- net at C26.1: now also C25.1, U7.6 (VDDCR); no longer C27.1
- net at R16.2: now also J26.7 (RD-), U7.22 (RXN)
- net at Y2.3: now also C28.1, U7.4 (XTAL2); no longer C31.1
- net CAN+: no longer names the net of U4.7 (CANH)
- net CAN+: now also R11.2, J8.1 (Pin_1)
- net CAN-: no longer names the net of U4.6 (CANL)
- net CAN-: now also R11.1, J8.2 (Pin_2)
- net LED2-INTSEL: no longer names the net of R18.1
- net LED2-INTSEL: now also U7.24 (RBIAS)
- net RX+: no longer names the net of R14.2
- net RX+: now also J26.2 (TD-), U7.20 (TXN)
- net RX-: no longer names the net of R15.2
- net RX-: now also J26.6 (RD+), U7.23 (RXP)
- net TX-: no longer names the net of R13.2
- net TX-: now also J26.1 (TD+), U7.21 (TXP)
- new net: R17.2, U7.10 (RXER/PHYAD0)
- new net: J26.12, R51.1, U7.2 (LED2/~{INTSEL})
- new net: J26.9, U7.3 (LED1/REGOFF)
- new net: J26.10, R52.1
- new net: J26.11, R53.1
Other:
- note added: "ETH"
- note removed: "ETH JACK"
- note removed: "ETH PHY"
- note removed: "Isolation is completely defeated if we use CAN"
- note removed: "The isolation on this board can only occur if we use an unshielded ethernet cable. For this reason, I think that connecting pins 13 and 14 to GND through a large isolation capacitor and bleed resistor might be a better choice."
