File: ali/v2/thermocouples/thermocouples.kicad_sch (KiCad schematic)
At the start: 4 parts

Commit message: mfw tcs
Other:
- added sheet CJC Sensors (cjc.kicad_sch)
- sheet Microcontroller ports: added CJC_~{RESET}, I2C4_SCL, I2C4_SDA; removed none

Commit message: Minor thermocouple updates
Other:
- sheet Microcontroller ports: added ADC_MISO, ADC_MOSI, ADC_SCLK, I2C1_SCL, I2C1_SDA; removed I2C4_SCL, I2C4_SDA, MISO, MOSI, SCLK
Changed lines of the file:
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@@
-			)
-		)
-		(pin "ADC_RESET" input
-			(at 165.1 142.24 0)
-			(effects
-				(font
-					(size 1.27 1.27)
-				)
-				(justify right)
 			)
 		)
@@
 			)
 		)
-		(pin "ADC_START" bidirectional
-			(at 165.1 139.7 0)
-			(effects
-				(font
-					(size 1.27 1.27)
-				)
-				(justify right)
-			)
-		)
 		(pin "FDCAN_RX" input
 			(at 101.6 157.48 180)
@@
 			)
 		)
-		(pin "MISO" input
-			(at 165.1 130.81 0)
-			(effects
-				(font
-					(size 1.27 1.27)
-				)
-				(justify right)
-			)
-		)
-		(pin "SCLK" output
-			(at 165.1 125.73 0)
-			(effects
-				(font
-					(size 1.27 1.27)
-				)
-				(justify right)
-			)
-		)
 		(pin "ETH_CRS_DV" input
 			(at 101.6 140.97 180)
@@
 			)
 		)
-		(pin "ADC_DRDY" input
+		(pin "ADC_DRDY" output
 			(at 165.1 137.16 0)
 			(effects
@@
 			)
 		)
-		(pin "MOSI" output
-			(at 165.1 128.27 0)
-			(effects
-				(font
-					(size 1.27 1.27)
-				)
-				(justify right)
-			)
-		)
 		(pin "ETH_~{RST}" output
 			(at 101.6 148.59 180)
@@
 			)
 		)
-		(pin "I2C4_SCL" bidirectional
+		(pin "CJC_~{RESET}" output
+			(at 165.1 158.75 0)
+			(effects
+				(font
+					(size 1.27 1.27)
+				)
+				(justify right)
+			)
+		)
+		(pin "I2C1_SDA" bidirectional
+			(at 165.1 156.21 0)
+			(effects
+				(font
+					(size 1.27 1.27)
+				)
+				(justify right)
+			)
+		)
+		(pin "ADC_START" output
+			(at 165.1 139.7 0)
+			(effects
+				(font
+					(size 1.27 1.27)
+				)
+				(justify right)
+			)
+		)
+		(pin "I2C1_SCL" bidirectional
 			(at 165.1 153.67 0)
 			(effects
@@
 			)
 		)
-		(pin "I2C4_SDA" bidirectional
-			(at 165.1 156.21 0)
+		(pin "ADC_RESET" output
+			(at 165.1 142.24 0)
 			(effects
 				(font
@@
 			)
 		)
-		(pin "CJC_~{RESET}" output
-			(at 165.1 158.75 0)
+		(pin "ADC_MISO" input
+			(at 165.1 130.81 0)
 			(effects
 				(font
+					(size 1.27 1.27)
+				)
+				(justify right)
+			)
+		)
+		(pin "ADC_MOSI" output
+			(at 165.1 128.27 0)
+			(effects
+				(font
+					(size 1.27 1.27)
+				)
+				(justify right)
+			)
+		)
+		(pin "ADC_SCLK" output
+			(at 165.1 125.73 0)
+			(effects
+				(font

Commit message: Begin prep for second board review
Other:
- sheet CJC Sensors ports: added none; removed ~{RESET}
- sheet Microcontroller ports: added none; removed CJC_~{RESET}
Changed lines of the file:
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@@
 	(paper "USLetter")
 	(title_block
-		(date "2026-09-11")
+		(date "2026-10-10")
 		(rev "1A")
 	)
@@
 	(wire
 		(pts
-			(xy 165.1 158.75) (xy 170.18 158.75)
-		)
-		(stroke
-			(width 0)
-			(type default)
-		)
-	)
-	(wire
-		(pts
 			(xy 165.1 130.81) (xy 170.18 130.81)
 		)
@@
 			)
 		)
-		(pin "CJC_~{RESET}" output
-			(at 165.1 158.75 0)
-			(effects
-				(font
-					(size 1.27 1.27)
-				)
-				(justify right)
-			)
-		)
 		(pin "I2C1_SDA" bidirectional
 			(at 165.1 156.21 0)
@@
 			(effects
 				(font
-					(size 1.27 1.27)
-				)
-				(justify left)
-			)
-		)
-		(pin "~{RESET}" input
-			(at 170.18 158.75 180)
-			(effects
-				(font
