File: ali/v2/pressuretransducers/connectivity.kicad_sch (KiCad schematic)
At the start: 27 parts, among them J7 Conn_01x03, J8 Vertical Ethernet, U3 TJA1462ATK, U4 LAN8742AI, Y2 25 MHz

Commit message: mfw pts
Parts:
- renumbered J7 to J6, J8 to J7

Commit message: Minor updates
Parts:
- renumbered C18 to C19, C19 to C20, C20 to C21, C21 to C22, C22 to C23, C23 to C24, C24 to C25, C25 to C26, C26 to C27, C27 to C28, C28 to C29, J6 to J8, J7 to J9, Y2 to Y3
