File: ali/v2/pressuretransducers/microcontroller.kicad_sch (KiCad schematic)
At the start: 45 parts, among them J1 Conn_02x01, J2 Conn_01x05, J3 USB_C_Receptacle_USB2.0_16P, J4 Conn_01x15, J5 Conn_02x09_Counter_Clockwise, J6 Screw_Terminal_01x02, SW1 SKRPANE010, U1 STM32H563RIV6, U2 UCC33420-Q1, U3 AP2112K-3.3, Y1 25 MHz

Commit message: mfw pts
Parts:
- removed C12: 22uF, APRL_Passive:C_0805, symbol Device:C_Small
- removed C13, C14: 10nF, APRL_Passive:C_0603, symbol Device:C_Small
- removed J4: Conn_01x15, APRL_Connector_Molex:Molex_CLIK-Mate_503159-1501_1x15-1MP_P1.50mm_Vertical, symbol Connector_Generic:Conn_01x15
- removed J5: Conn_02x09_Counter_Clockwise, Connector_IDC:IDC-Header_2x09_P2.54mm_Vertical, symbol Connector_Generic:Conn_02x09_Odd_Even
- removed U2: UCC33420-Q1, APRL_Package_QFN:VSON-12_4x5mm_P0.65mm, symbol APRL_Power:UCC33420
- added F2: 750mA, APRL_Passive:Fuse_1812_4532Metric, symbol Device:Fuse_Small
- added J24: Conn_02x09_Counter_Clockwise, Connector_IDC:IDC-Header_2x09_P2.54mm_Vertical, symbol Connector_Generic:Conn_02x09_Odd_Even
- added J25: Conn_01x15, APRL_Connector_Molex:Molex_CLIK-Mate_503159-1501_1x15-1MP_P1.50mm_Vertical, symbol Connector_Generic:Conn_01x15
- added J4: Screw_Terminal_01x02, Connector_Phoenix_MSTB:PhoenixContact_MSTBV_2,5_2-GF-5,08_1x02_P5.08mm_Vertical_ThreadedFlange_MountHole, symbol Connector:Screw_Terminal_01x02
- U2: renamed from U3; MANUFACTURER Didoes Inc. -> Diodes Inc.
- renumbered C15 to C12, C16 to C13, C17 to C14, C18 to C15, C19 to C16, C20 to C17, D4 to D1, D5 to D2, D1 to D3, D2 to D4, D3 to D5, F2 to F3, J6 to J5, R4 to R3, R5 to R4, R3 to R5
Connections:
- net Earth is gone; now on net GND: J5.1 (Pin_1)
- net +3.3V: now also J24.2 (Pin_2), J25.5 (Pin_5)
- net +5V: now also F3.2, J24.1 (Pin_1), J25.6 (Pin_6)
- net GND: now also J24.10 (Pin_10), J24.12 (Pin_12), J24.14 (Pin_14), J24.16 (Pin_16), J24.18 (Pin_18), J24.4 (Pin_4), J24.6 (Pin_6), J24.8 (Pin_8), J25.2 (Pin_2), J4.1 (Pin_1)
- net PA15: now also J25.15 (Pin_15)
- net PA3: now also J24.17 (Pin_17)
- net PA4: now also J24.15 (Pin_15)
- net PA5: now also J24.13 (Pin_13)
- net PA6: now also J24.11 (Pin_11)
- net PB10: now also J24.3 (Pin_3)
- net USER_LED_1: now also U1.39 (PD12); no longer U1.26 (PB0)
- net USER_LED_2: now also U1.40 (PC6); no longer U1.27 (PB1)
- net USER_LED_3: now also U1.41 (PC7); no longer U1.28 (PB2)
- net ADC1_DRDY: now reaches U1.2 (PC13)
- net ADC1_~{RST}: now reaches U1.4 (PC15)
- net ADC_CS renamed I2C1_SCL
- net I2C1_SCL: now also J25.8 (Pin_8)
- net ADC_DRDY renamed SPI3_MOSI
- net SPI3_MOSI: now also J25.12 (Pin_12)
- net ADC_RESET renamed SPI3_MISO
- net SPI3_MISO: now also J25.13 (Pin_13)
- net ADC_START renamed I2C1_SDA
- net I2C1_SDA: now also J25.7 (Pin_7)
- net CJC_~{RESET} renamed ADC2_DRDY
- net I2C4_SCL renamed UART4_RX
- net UART4_RX: now also J25.4 (Pin_4)
- net I2C4_SDA renamed UART4_TX
- net UART4_TX: now also J25.3 (Pin_3)
- net MISO renamed SPI1_MISO
- net SPI1_MISO: now also J25.10 (Pin_10)
- net MOSI renamed SPI1_MOSI
- net SPI1_MOSI: now also J25.9 (Pin_9)
- net PA9: no longer names the net of U1.45 (PA9)
- net PC10 renamed SPI3_SCK
- net SPI3_SCK: now also J25.14 (Pin_14)
- net PC14 renamed ADC1_CS
- net PC2 renamed ADC2_~{RST}
- net PC3 renamed ADC2_CS
- net PE0: no longer names the net of U1.65 (PE0)
- net SCLK renamed SPI1_SCK
- net SPI1_SCK: now also J25.11 (Pin_11)
- new net: F2.2, J4.2 (Pin_2)
- new net +24V: F2.1, J25.1 (Pin_1)
- new net PB0: J24.9 (Pin_9), U1.26 (PB0)
- new net PB1: J24.7 (Pin_7), U1.27 (PB1)
- new net PB2: J24.5 (Pin_5), U1.28 (PB2)
- no-connect marks 17 -> 14
Other:
- note added: "not sure if this is too much for OC, I don't think a singlular TVS diode (which is the case I want to protect against) is enough for this"
- note removed: "Expansion Port (for adding more peripherals)"
- note removed: "Spare GPIO"
- note removed: "chip has a weird footprint in stock at lcsc btw"
- note removed: "fsw is 64.5 MHz (which is kinda crazy) I wasn't able to find a bead thats a good fit so it is what it is"
- moved on the sheet: C12, C13, C14, C15, C16, C17, D1, D2, D3, D4, D5, F1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
Changed lines of the file:
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@@
 	(title_block
 		(date "2026-09-11")
-		(rev "1A")
 	)

Commit message: Minor updates
Parts:
- removed J25: Conn_01x15, APRL_Connector_Molex:Molex_CLIK-Mate_503159-1501_1x15-1MP_P1.50mm_Vertical, symbol Connector_Generic:Conn_01x15
- added C18: 100nF, APRL_Passive:C_0603, symbol Device:C_Small
- added J4: Conn_01x15, APRL_Connector_Molex:Molex_CLIK-Mate_503159-1501_1x15-1MP_P1.50mm_Vertical, symbol Connector_Generic:Conn_01x15
- added Y2: 8.192 MHz, APRL_Passive:Oscillator_SCTF_SX3M_3.2x2.5mm, symbol APRL_Misc:SX3M-xxxMHz
- renumbered F3 to F2, F2 to F3, J24 to J5, J5 to J6, J4 to J7
Connections:
- net ADC2_DRDY is gone; now on net ADC2_CS: U1.8 (PC0)
- net +3.3V: now also C18.1, J4.12 (Pin_12), Y2.1 (EN), Y2.4 (Vdd)
- net +5V: now also J4.1 (Pin_1)
- net ADC2_CS: no longer U1.11 (PC3)
- net GND: now also C18.2, J4.2 (Pin_2), Y2.2 (GND)
- net I2C1_SCL: now also J4.8 (Pin_8)
- net I2C1_SDA: now also J4.7 (Pin_7)
- net PA6: now also J5.13 (Pin_13); no longer J5.11 (Pin_11)
- net PB0: now also J5.11 (Pin_11); no longer J5.9 (Pin_9)
- net PB1: now also J5.9 (Pin_9); no longer J5.7 (Pin_7)
- net PB2: now also J5.7 (Pin_7); no longer J5.5 (Pin_5)
- net UART4_RX: now also J4.6 (Pin_6)
- net UART4_TX: now also J4.5 (Pin_5)
- net USER_LED_1: now also U1.40 (PC6); no longer U1.39 (PD12)
- net USER_LED_2: now also U1.41 (PC7); no longer U1.40 (PC6)
- net USER_LED_3: now also U1.42 (PC8); no longer U1.41 (PC7)
- net PD11: now reaches U1.38 (PD11)
- net PD11: now also J5.5 (Pin_5)
- net ADC1_DRDY renamed PC13
- net PC13: now also J4.3 (Pin_3)
- net ADC1_~{RST} renamed ADC_RESET
- net ADC_RESET: now also J4.4 (Pin_4)
- net ADC2_~{RST}: no longer names the net of U1.10 (PC2)
- net PA15 renamed TIM2_CH1
- net TIM2_CH1: now also J4.14 (Pin_14)
- net PA3 renamed TIM2_CH4
- net PA5 renamed ADC_SCLK
- net ADC_SCLK: now also J4.9 (Pin_9); no longer J5.13 (Pin_13)
- net PB10 renamed PD12
- net PD12: now also U1.39 (PD12); no longer U1.29 (PB10)
- net SPI1_MISO renamed ADC_MISO
- net ADC_MISO: now also J4.10 (Pin_10)
- net SPI1_MOSI renamed ADC_MOSI
- net ADC_MOSI: now also J4.11 (Pin_11)
- net SPI1_SCK renamed ADC_DRDY
- net SPI3_MISO: no longer names the net of U1.55 (PC11)
- net SPI3_MOSI renamed PC12
- net PC12: now also J4.13 (Pin_13)
- net SPI3_SCK: no longer names the net of U1.54 (PC10)
- new net ADC_CLK: Y2.3 (OUT)
- new net TIM2_CH3: J4.15 (Pin_15), U1.29 (PB10)
- no-connect marks 14 -> 16
Other:
- note added: "ADC OSC"
- moved on the sheet: C12, C13, C14, C15, C16, C17, F2, F3, J5, J6, J7, U2
