File: ali/v2/pressuretransducers/pressuretransducers.kicad_pcb (KiCad board)
At the start: 4 copper layers, 85 x 76 mm, 239 parts, among them J1 Conn_02x01, J10 Conn_01x02, J11 Conn_01x02, J12 Conn_01x02, J13 Conn_01x02, J14 Conn_01x02, J15 Conn_01x02, J16 Conn_01x02, J17 Conn_01x02, J18 Conn_01x02, J19 Conn_01x02, J2 Conn_01x05, J20 Conn_01x02, J21 Conn_01x02, J22 Conn_01x02, J23 Conn_01x02, J24 Conn_02x09_Counter_Clockwise, J25 Conn_01x15, J3 USB_C_Receptacle_USB2.0_16P, J4 Screw_Terminal_01x02, J5 Screw_Terminal_01x02, J6 Conn_01x03, J7 Vertical Ethernet, J8 Conn_01x02, J9 Conn_01x02, SW1 SKRPANE010, U1 STM32H563RIV6, U2 AP2112K-3.3, U3 TJA1462ATK, U4 LAN8742AI, U5 ADS131M08IRSN, U6 ADS131M08IRSN, Y1 25 MHz, Y2 25 MHz, Y3 8.192 MHz, Y4 8.192 MHz

Commit message: Minor updates
Parts:
- removed the C35 at (123.4, 75.8)
- removed the C36 at (127.9, 79.8)
- removed the C67 at (124.0, 105.2)
- removed the C68 at (127.8, 109.8)
- removed the Y3 at (126.6, 76.8)
- removed Y4: 8.192 MHz, APRL_Passive:3225-4P-L
- added C18: 100nF, APRL_Passive:C_0603, F.Cu at (125.5, 79.3)
- added Y2: 8.192 MHz, APRL_Passive:Oscillator_SCTF_SX3M_3.2x2.5mm, F.Cu at (128.0, 79.2)
- moved D3 4.40 mm to (162.3, 110.8)
- moved D4 4.40 mm to (162.3, 109.0)
- moved R5 4.40 mm to (159.1, 110.8)
- moved R6 4.40 mm to (159.1, 109.0)
- moved D5 4.40 mm to (162.3, 107.2)
- moved R7 4.40 mm to (159.1, 107.2)
- moved C6 0.20 mm to (149.2, 95.2)
- moved C8 0.20 mm to (138.3, 96.8)
- moved Y1 0.19 mm to (135.0, 95.0)
- renumbered C18 to C19, C19 to C20, C20 to C21, C21 to C22, C22 to C23, C23 to C24, C24 to C25, C25 to C26, C26 to C27, C27 to C28, C28 to C29, C37 to C30, C40 to C31, C39 to C32, C42 to C33, C38 to C34, C41 to C35, C29 to C36, C30 to C37, C31 to C38, C34 to C39, C32 to C40, C43 to C41, C46 to C42, C45 to C43, C48 to C44, C44 to C45, C47 to C46, C49 to C47, C52 to C48, C51 to C49, C54 to C50, C50 to C51, C53 to C52, C33 to C53, C55 to C54, C58 to C55, C57 to C56, C60 to C57, C56 to C58, C69 to C60, C72 to C61, C71 to C62, C74 to C63, C70 to C64, C73 to C65, C61 to C66, C62 to C67, C63 to C68, C66 to C69, C64 to C70, C75 to C71, C78 to C72, C77 to C73, C80 to C74, C76 to C75, C79 to C76, C81 to C77, C84 to C78, C83 to C79, C86 to C80, C82 to C81, C85 to C82, C65 to C83, C87 to C84, C90 to C85, C89 to C86, C92 to C87, C91 to C89, F3 to F2, F2 to F3, J8 to J10, J9 to J11, J10 to J12, J11 to J13, J12 to J14, J13 to J15, J14 to J16, J15 to J17, J16 to J18, J17 to J19, J18 to J20, J19 to J21, J20 to J22, J21 to J23, J22 to J24, J23 to J25, J25 to J4, J24 to J5, J5 to J6, J4 to J7, J6 to J8, J7 to J9, R20 to R19, R23 to R20, R19 to R21, R21 to R23, R26 to R25, R29 to R26, R25 to R27, R27 to R29, R32 to R31, R35 to R32, R31 to R33, R33 to R35, R38 to R37, R41 to R38, R37 to R39, R39 to R41, R44 to R43, R47 to R44, R43 to R45, R45 to R47, R50 to R49, R53 to R50, R49 to R51, R51 to R53, R56 to R55, R59 to R56, R55 to R57, R57 to R59, R62 to R61, R65 to R62, R61 to R63, R63 to R65, Y2 to Y3
Connections:
- net /Microcontroller/PA3 renamed /Microcontroller/TIM2_CH4
- J4 pad 1: +24V -> +5V
- J4 pad 11: /Analog 1/SCLK -> /Analog 1/MOSI
- J4 pad 12: /Microcontroller/SPI3_MOSI -> +3.3V
- J4 pad 13: /Microcontroller/SPI3_MISO -> /Microcontroller/PC12
- J4 pad 14: /Microcontroller/SPI3_SCK -> /Microcontroller/TIM2_CH1
- J4 pad 15: /Microcontroller/PA15 -> /Microcontroller/TIM2_CH3
- J4 pad 3: /Microcontroller/UART4_TX -> /Microcontroller/PC13
- J4 pad 4: /Microcontroller/UART4_RX -> /Analog 1/RESET
- J4 pad 5: +3.3V -> /Microcontroller/UART4_TX
- J4 pad 6: +5V -> /Microcontroller/UART4_RX
- J4 pad 9: /Analog 1/MOSI -> /Analog 1/SCLK
- J5 pad 11: /Microcontroller/PA6 -> /Microcontroller/PB0
- J5 pad 13: /Microcontroller/PA5 -> /Microcontroller/PA6
- J5 pad 3: /Microcontroller/PB10 -> /Microcontroller/PD12
- J5 pad 5: /Microcontroller/PB2 -> /Microcontroller/PD11
- J5 pad 7: /Microcontroller/PB1 -> /Microcontroller/PB2
- J5 pad 9: /Microcontroller/PB0 -> /Microcontroller/PB1
- U1 pad 10: /Analog 2/RESET -> unconnected-(U1-PC2-Pad10)
- U1 pad 11: /Analog 2/CS -> unconnected-(U1-PC3-Pad11)
- U1 pad 2: /Analog 1/DRDY -> /Microcontroller/PC13
- U1 pad 21: /Microcontroller/PA5 -> /Analog 1/SCLK
- U1 pad 29: /Microcontroller/PB10 -> /Microcontroller/TIM2_CH3
- U1 pad 38: unconnected-(U1-PD11-Pad38) -> /Microcontroller/PD11
- U1 pad 39: /Microcontroller/USER_LED_1 -> /Microcontroller/PD12
- U1 pad 40: /Microcontroller/USER_LED_2 -> /Microcontroller/USER_LED_1
- U1 pad 41: /Microcontroller/USER_LED_3 -> /Microcontroller/USER_LED_2
- U1 pad 42: unconnected-(U1-PC8-Pad42) -> /Microcontroller/USER_LED_3
- U1 pad 53: /Microcontroller/PA15 -> /Microcontroller/TIM2_CH1
- U1 pad 54: /Microcontroller/SPI3_SCK -> unconnected-(U1-PC10-Pad54)
- U1 pad 55: /Microcontroller/SPI3_MISO -> unconnected-(U1-PC11-Pad55)
- U1 pad 56: /Microcontroller/SPI3_MOSI -> /Microcontroller/PC12
- U1 pad 57: /Analog 1/SCLK -> /Analog 1/DRDY
- U1 pad 8: /Analog 2/DRDY -> /Analog 2/CS
- U5 pad 22: Net-(U5-XTAL2) -> unconnected-(U5-XTAL2-Pad22)
- U5 pad 23: Net-(U5-XTAL1/CLKIN) -> /Analog 1/CLK
- U6 pad 16: /Analog 2/RESET -> /Analog 1/RESET
- U6 pad 22: Net-(U6-XTAL2) -> unconnected-(U6-XTAL2-Pad22)
- U6 pad 23: Net-(U6-XTAL1/CLKIN) -> /Analog 1/CLK
Routing:
- net /Analog 1/RESET: track 20.2 -> 80.1 mm, vias 0 -> 4
- net /Microcontroller/TIM2_CH3: track 0.00 -> 53.6 mm, vias 0 -> 3
- net /Microcontroller/PD12: track 0.00 -> 50.7 mm, vias 0 -> 1
- net /Microcontroller/PD11: track 0.00 -> 49.5 mm, vias 0 -> 1
- net /Microcontroller/PB10: track 44.6 -> 0.00 mm, vias 1 -> 0
- net /Microcontroller/PA5: track 42.3 -> 0.00 mm, vias 2 -> 0
- net /Analog 1/CLK: track 0.00 -> 40.5 mm, vias 0 -> 2
- net /Microcontroller/TIM2_CH1: track 0.00 -> 40.2 mm
- net /Microcontroller/SPI3_SCK: track 40.0 -> 0.00 mm
- net /Microcontroller/PA15: track 38.7 -> 0.00 mm
- net /Microcontroller/SPI3_MOSI: track 38.4 -> 0.00 mm
- net /Microcontroller/SPI3_MISO: track 37.1 -> 0.00 mm
- net /Microcontroller/PC12: track 0.00 -> 37.0 mm
- net /Analog 2/RESET: track 33.8 -> 0.00 mm, vias 2 -> 0
- net /Microcontroller/PC13: track 0.00 -> 33.0 mm, vias 0 -> 2
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
Commit message: Swap to sync'd ADS1261s on LC, update README and clean up Just scripts, some frame changes too.
Other:
- board text added: "REV ${REV}"
- board text removed: "REV 2A"
