File: ali/v2/pressuretransducers/analog.kicad_sch (KiCad schematic)
At the start: 79 parts, among them J10 Conn_01x02, J11 Conn_01x02, J12 Conn_01x02, J13 Conn_01x02, J14 Conn_01x02, J15 Conn_01x02, J16 Conn_01x02, J17 Conn_01x02, U5 ADS131M08IRSN

Commit message: Begin prep for second board review
Parts:
- removed C31, C34, C45, C46, C47, C48, C51, C52, C54, C55, C59: 1nF, APRL_Passive:C_0603, symbol Device:C_Small
- removed C32, C33, C43, C44, C49, C56, C57: 10nF, APRL_Passive:C_0603, symbol Device:C_Small
- removed C40: 100nF, APRL_Passive:C_0603, symbol Device:C_Small
- removed D6: SMF7V0A, Diode_SMD:D_SMF, symbol Device:D_Zener_Small_Filled
- removed J10: Conn_01x02, APRL_Connector_Molex:Molex_CLIK-Mate_503159-0201_1x02-1MP_P1.50mm_Vertical, symbol Connector_Generic:Conn_01x02
- removed NT1, NT2, NT3, NT4, NT5, NT6, NT7, NT8: NetTie_2, APRL_Misc:NetTie-2_SMD_Pad0.15mm, symbol Device:NetTie_2
- removed R35, R36, R41: 47.5R, APRL_Passive:R_0805, symbol Device:R_Small_US
- removed R37, R38, R39, R43, R44: 1k, APRL_Passive:R_0603, symbol Device:R_Small_US
- added C29, C37, C38, C39: 1nF, APRL_Passive:C_0603, symbol Device:C_Small
- added C36: 12pF, APRL_Passive:C_0603, symbol Device:C_Small
- added D13: VTVS3V3ASMF, Diode_SMD:D_SMF, symbol Device:D_Zener_Small_Filled
- added F10, F4, F6, F8: 100mA, APRL_Passive:Fuse_1206_3216Metric, symbol Device:Fuse_Small
- added J17: Conn_01x02, APRL_Connector_Molex:Molex_CLIK-Mate_503159-0201_1x02-1MP_P1.50mm_Vertical, symbol Connector_Generic:Conn_01x02
- added Y3: 8.192 MHz, APRL_Passive:3225-4P-L, symbol Device:Crystal_GND24
- C50: value 10nF -> 100nF; MPN GRM1885C1H103JA01 -> GRM188R72A104KA35
- C58: value 1nF -> 12pF; MPN GRM1885C1H102FA01 -> GRM1885C1H120JA01
- D10, D11, D12, D7, D8, D9: value SMF7V0A -> VTVS3V3ASMF; MPN SMF7V0A-E3-18 -> VTVS3V3ASMF-M3-08
- D6: renamed from D13; value SMF7V0A -> VTVS3V3ASMF; MPN SMF7V0A-E3-18 -> VTVS3V3ASMF-M3-08
- R22, R26, R28, R32, R34: value 1k -> 47.5R; footprint APRL_Passive:R_0603 -> APRL_Passive:R_0805; MANUFACTURER Yageo -> RESI; MPN RT0603BRD071KL -> ERA-6AEB47R5V
- R23, R29: value 47.5R -> 1k; footprint APRL_Passive:R_0805 -> APRL_Passive:R_0603; MANUFACTURER RESI -> Yageo; MPN ERA-6AEB47R5V -> RT0603BRD071KL
- renumbered C36 to C31, C37 to C32, C38 to C33, C39 to C34, C53 to C40, J17 to J10, R40 to R19, R42 to R20
Connections:
- net AIN3- is gone; now on net GND: R32.2, U5.3 (AIN3N)
- net AIN4- is gone; now on net GND: U5.6 (AIN4N)
- net AIN6+ is gone; now on an unnamed net: U5.9 (AIN6P)
- net AIN6- is gone; now on net GND: C58.2, U5.10 (AIN6N)
- net AIN7- is gone; now on net GND: U5.11 (AIN7N)
- net +24V: now also F10.2, F4.2, F6.2, F8.2; no longer J10.2 (Pin_2), J11.2 (Pin_2), J12.2 (Pin_2), J13.2 (Pin_2), J14.2 (Pin_2), J15.2 (Pin_2), J16.2 (Pin_2)
- net GND: now also C30.1, C41.1, C42.1, C50.2, R22.2, R26.2, R28.2, R34.2, U5.2 (AIN2N), U5.30 (AIN0N), U5.31 (AIN1N), U5.7 (AIN5N), C29.1, C36.2, C37.1, C38.1, C39.1, D13.2 (A), Y3.2 (G), Y3.4 (G); no longer C30.2, C41.2, C42.2, C58.1, R23.2, R29.2
- net at D12.1 (K), J16.1 (Pin_1): now also R31.1, R32.1
- net at D10.1 (K), J14.1 (Pin_1): now also R27.1, R28.1; no longer R33.1
- net at D8.1 (K), J12.1 (Pin_1): now also R23.1, R24.1; no longer R27.1, R29.1
- net at R21.1: now also D7.1 (K), J11.1 (Pin_1), R22.1; no longer R23.1
- net at D11.1 (K), J15.1 (Pin_1): now also R29.1, R30.1; no longer R34.1
- net at D9.1 (K), J13.1 (Pin_1): now also R25.1, R26.1; no longer R28.1, R30.1
- net at U5.14 (REFIN): now also C50.1
- net at U5.22 (XTAL2): now also C58.1, Y3.3
- removed net AIN0+: C30.1, R21.2, U5.29 (AIN0P)
- net AIN0-: no longer names the net of R25.2
- net AIN0-: now also U5.4 (AIN3P), C37.2; no longer U5.30 (AIN0N)
- net AIN1+: no longer names the net of U5.32 (AIN1P)
- net AIN1+: now also C30.2, R21.2; no longer R22.2
- removed net AIN1-: C35.2, R26.2, U5.31 (AIN1N)
- removed net AIN2+: C41.1, R27.2, U5.1 (AIN2P)
- net AIN2-: no longer names the net of R31.2
- net AIN2-: now also C41.2; no longer U5.2 (AIN2N)
- removed net AIN3+: C42.1, R28.2, U5.4 (AIN3P)
- net AIN4+: no longer names the net of R33.2
- net AIN4+: now also C42.2, U5.12 (AIN7P); no longer U5.5 (AIN4P)
- removed net AIN5+: C50.2, R34.2, U5.8 (AIN5P)
- removed net AIN5-: C50.1, U5.7 (AIN5N)
- net AIN7+: no longer names the net of R19.2
- net AIN7+: now also U5.29 (AIN0P), C29.2; no longer U5.12 (AIN7P)
- net CLK: no longer names the net of U5.23 (XTAL1/CLKIN)
- net CLK: now also C36.1, Y3.1
- new net: F6.1, J12.2 (Pin_2), J13.2 (Pin_2)
- new net: F4.1, J10.2 (Pin_2), J11.2 (Pin_2)
- new net: D13.1 (K), J17.1 (Pin_1), R33.1, R34.1
- new net: C35.2, R23.2, U5.1 (AIN2P)
- new net: F8.1, J14.2 (Pin_2), J15.2 (Pin_2)
- new net: C38.2, R27.2, U5.5 (AIN4P)
- new net: C39.2, R29.2, U5.8 (AIN5P)
- new net: F10.1, J16.2 (Pin_2), J17.2 (Pin_2)
- no-connect marks 1 -> 0
Other:
- note removed: "ADC"
- note removed: "INPUTS"
- note removed: "It would be trivial to isolate this entire board using the same trick we used on the thermocouple board, where we just place a dc/dc isolator chip on the +5V rail. This would enhance the protection of our system by allowing us to isolate +24V, which would prevent ground bounce and greatly limit damage from shorts because there is no return line back to the power supply if its ground is floating. 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"
- note removed: "On this board in particular the CM caps are not required, but we can always mark them DNP and they shouldn't pose any problems"
- note removed: "The idea behind the net ties is to create a kelvin connection but I don't think I'm really achieving it here and I don't think that it'd actually help if I did"
- note removed: "The protection diode and shunt resistor are going to immediately blow and/or short if this thing actually got shorted, but I'm not sure if we want a PTC on every input, especially since it'd mean there'd be a nontrivial change in DC resistance relative to the shunt. That being said, it shouldn't affect us if we placed it on the high side, though."
- note removed: "The voltage drop over these 1K resistors is nontrivial but can be calibrated out"
- note removed: "These caps are all c0g and these resistors are all thin film. I started placing MPN and Manufacturer on the fields of nearly every part on these boards so that we can standardize on certain parts and to make ordering easier, and to prevent the TC situation where we used X5Rs for the DM filtering on the AFE"
- note removed: "These connectors were colored by claude which is why they're off I did search for connectors that are not just gray but they simply do not exist"
- note removed: "fcm = 159 kHz fdm = 7.58 kHz"
- moved on the sheet: C31, C32, C33, C34, C40, D6, J10, R19, R20, U5
