File: ali/v2/valvedrivers/valvedrivers.kicad_pcb (KiCad board)
At the start: 4 copper layers, 85 x 76 mm, 152 parts, among them J1 Conn_02x01, J10 Conn_01x02, J11 Conn_01x02, J12 Conn_01x02, J13 Conn_01x02, J14 Conn_01x02, J15 Conn_01x02, J16 Conn_01x02, J17 Conn_01x02, J18 Conn_01x02, J19 Conn_01x02, J2 Conn_01x05, J20 Conn_01x02, J3 USB_C_Receptacle_USB2.0_16P, J4 Screw_Terminal_01x02, J5 Screw_Terminal_01x02, J6 Screw_Terminal_01x02, J7 Conn_01x03, J8 Vertical Ethernet, J9 Conn_01x02, SW1 SKRPANE010, U1 STM32H563RIV6, U10 PS2841-4B, U11 PS2841-4B, U12 IPS4140HQ, U13 PS2841-4B, U14 PS2841-4B, U2 LTV-816S, U3 AP2112K-3.3, U4 TJA1462ATK, U5 LAN8742AI, U6 IPS4140HQ, U7 PS2841-4B, U8 PS2841-4B, U9 IPS4140HQ, Y1 25 MHz, Y2 25 MHz

Commit message: Small stuff
Parts:
- U1: footprint Package_DFN_QFN:QFN-68-1EP_8x8mm_P0.4mm_EP6.4x6.4mm -> APRL_Package_QFN:QFN-68-1EP_8x8mm_P0.4mm_EP6.4x6.4mm
- moved C1 0.50 mm to (149.5, 93.7)
- moved C6 0.50 mm to (149.5, 95.2)
Routing:
- net +24V: track 66.3 -> 70.7 mm
- net /Connectivity/ETH_MDIO: track 26.1 -> 26.8 mm
- net /Drivers 2/IN3: track 13.1 -> 13.8 mm
- net GNDPWR: vias 184 -> 228

Commit message: Swap to sync'd ADS1261s on LC, update README and clean up Just scripts, some frame changes too.
Other:
- board text added: "REV ${REV}"
- board text removed: "REV 2A"

Commit message: Fix ERC issues
Parts:
- U1: footprint APRL_Package_QFN:QFN-68-1EP_8x8mm_P0.4mm_EP6.4x6.4mm -> Package_DFN_QFN:QFN-68-1EP_8x8mm_P0.4mm_EP6.4x6.4mm

Commit message: Idk why this package change keeps happening
Parts:
- U1: footprint Package_DFN_QFN:QFN-68-1EP_8x8mm_P0.4mm_EP6.4x6.4mm -> APRL_Package_QFN:QFN-68-1EP_8x8mm_P0.4mm_EP6.4x6.4mm
Changed lines of the file:
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@@
 		)
 	)
-	(footprint "Package_DFN_QFN:QFN-68-1EP_8x8mm_P0.4mm_EP6.4x6.4mm"
+	(footprint "APRL_Package_QFN:QFN-68-1EP_8x8mm_P0.4mm_EP6.4x6.4mm"
 		(layer "F.Cu")
 		(at 145.7125 98.925)
@@
 		(pad "" smd roundrect
 			(at -2.4 -2.4)
-			(size 1.29 1.29)
+			(size 1.42 1.42)
 			(layers "F.Paste")
 			(roundrect_rratio 0.193798)
@@
 		(pad "" smd roundrect
 			(at -2.4 -0.8)
-			(size 1.29 1.29)
+			(size 1.42 1.42)
 			(layers "F.Paste")
 			(roundrect_rratio 0.193798)
@@
 		(pad "" smd roundrect
 			(at -2.4 0.8)
-			(size 1.29 1.29)
+			(size 1.42 1.42)
 			(layers "F.Paste")
 			(roundrect_rratio 0.193798)
@@
 		(pad "" smd roundrect
 			(at -2.4 2.4)
-			(size 1.29 1.29)
+			(size 1.42 1.42)
 			(layers "F.Paste")
 			(roundrect_rratio 0.193798)
@@
 		(pad "" smd roundrect
 			(at -0.8 -2.4)
-			(size 1.29 1.29)
+			(size 1.42 1.42)
 			(layers "F.Paste")
 			(roundrect_rratio 0.193798)
@@
 		(pad "" smd roundrect
 			(at -0.8 -0.8)
-			(size 1.29 1.29)
+			(size 1.42 1.42)
 			(layers "F.Paste")
 			(roundrect_rratio 0.193798)
@@
 		(pad "" smd roundrect
 			(at -0.8 0.8)
-			(size 1.29 1.29)
+			(size 1.42 1.42)
 			(layers "F.Paste")
 			(roundrect_rratio 0.193798)
@@
 		(pad "" smd roundrect
 			(at -0.8 2.4)
-			(size 1.29 1.29)
+			(size 1.42 1.42)
 			(layers "F.Paste")
 			(roundrect_rratio 0.193798)
@@
 		(pad "" smd roundrect
 			(at 0.8 -2.4)
-			(size 1.29 1.29)
+			(size 1.42 1.42)
 			(layers "F.Paste")
 			(roundrect_rratio 0.193798)
@@
 		(pad "" smd roundrect
 			(at 0.8 -0.8)
-			(size 1.29 1.29)
+			(size 1.42 1.42)
 			(layers "F.Paste")
 			(roundrect_rratio 0.193798)
@@
 		(pad "" smd roundrect
 			(at 0.8 0.8)
-			(size 1.29 1.29)
+			(size 1.42 1.42)
 			(layers "F.Paste")
 			(roundrect_rratio 0.193798)
@@
 		(pad "" smd roundrect
 			(at 0.8 2.4)
-			(size 1.29 1.29)
+			(size 1.42 1.42)
 			(layers "F.Paste")
 			(roundrect_rratio 0.193798)
@@
 		(pad "" smd roundrect
 			(at 2.4 -2.4)
-			(size 1.29 1.29)
+			(size 1.42 1.42)
 			(layers "F.Paste")
 			(roundrect_rratio 0.193798)
@@
 		(pad "" smd roundrect
 			(at 2.4 -0.8)
-			(size 1.29 1.29)
+			(size 1.42 1.42)
 			(layers "F.Paste")
 			(roundrect_rratio 0.193798)
@@
 		(pad "" smd roundrect
 			(at 2.4 0.8)
-			(size 1.29 1.29)
+			(size 1.42 1.42)
 			(layers "F.Paste")
 			(roundrect_rratio 0.193798)
@@
 		(pad "" smd roundrect
 			(at 2.4 2.4)
-			(size 1.29 1.29)
+			(size 1.42 1.42)
 			(layers "F.Paste")
 			(roundrect_rratio 0.193798)
@@
 			(pinfunction "VDD_68")
 			(pintype "power_in")
+		)
+		(pad "69" thru_hole circle
+			(at -2.8 -2.8 90)
+			(size 0.5 0.5)
+			(drill 0.3)
+			(layers "*.Cu")
+			(remove_unused_layers no)
+			(net "GND")
+			(pinfunction "VSS_69")
+			(pintype "passive")
+		)
+		(pad "69" thru_hole circle
+			(at -2.8 -1.68 90)
+			(size 0.5 0.5)
+			(drill 0.3)
+			(layers "*.Cu")
+			(remove_unused_layers no)
+			(net "GND")
+			(pinfunction "VSS_69")
+			(pintype "passive")
+		)
+		(pad "69" thru_hole circle
+			(at -2.8 -0.56 90)
+			(size 0.5 0.5)
+			(drill 0.3)
+			(layers "*.Cu")
+			(remove_unused_layers no)
+			(net "GND")
+			(pinfunction "VSS_69")
+			(pintype "passive")
+		)
+		(pad "69" thru_hole circle
+			(at -2.8 0.56 90)
+			(size 0.5 0.5)
+			(drill 0.3)
+			(layers "*.Cu")
+			(remove_unused_layers no)
+			(net "GND")
+			(pinfunction "VSS_69")
+			(pintype "passive")
+		)
+		(pad "69" thru_hole circle
+			(at -2.8 1.68 90)
+			(size 0.5 0.5)
+			(drill 0.3)
+			(layers "*.Cu")
+			(remove_unused_layers no)
+			(net "GND")
+			(pinfunction "VSS_69")
+			(pintype "passive")
+		)
+		(pad "69" thru_hole circle
+			(at -2.8 2.8 90)
+			(size 0.5 0.5)
+			(drill 0.3)
+			(property pad_prop_heatsink)
+			(layers "*.Cu")
+			(remove_unused_layers no)
+			(net "GND")
+			(pinfunction "VSS_69")
+			(pintype "passive")
+		)
+		(pad "69" thru_hole circle
+			(at -1.68 -2.8)
+			(size 0.5 0.5)
+			(drill 0.3)
+			(layers "*.Cu")
+			(remove_unused_layers no)
+			(net "GND")
+			(pinfunction "VSS_69")
+			(pintype "passive")
+		)
+		(pad "69" thru_hole circle
+			(at -1.68 2.8 180)
+			(size 0.5 0.5)
+			(drill 0.3)
+			(layers "*.Cu")
+			(remove_unused_layers no)
+			(net "GND")
+			(pinfunction "VSS_69")
+			(pintype "passive")
+		)
+		(pad "69" thru_hole circle
+			(at -0.56 -2.8)
+			(size 0.5 0.5)
+			(drill 0.3)
+			(layers "*.Cu")
+			(remove_unused_layers no)
+			(net "GND")
+			(pinfunction "VSS_69")
+			(pintype "passive")
+		)
+		(pad "69" thru_hole circle
+			(at -0.56 2.8 180)
+			(size 0.5 0.5)
+			(drill 0.3)
+			(layers "*.Cu")
+			(remove_unused_layers no)
+			(net "GND")
+			(pinfunction "VSS_69")
+			(pintype "passive")
 		)
 		(pad "69" smd rect
@@
 			(zone_connect 2)
 		)
+		(pad "69" thru_hole circle
+			(at 0.56 -2.8)
+			(size 0.5 0.5)
+			(drill 0.3)
+			(layers "*.Cu")
+			(remove_unused_layers no)
+			(net "GND")
+			(pinfunction "VSS_69")
+			(pintype "passive")
+		)
+		(pad "69" thru_hole circle
+			(at 0.56 2.8 180)
+			(size 0.5 0.5)
+			(drill 0.3)
+			(layers "*.Cu")
+			(remove_unused_layers no)
+			(net "GND")
+			(pinfunction "VSS_69")
+			(pintype "passive")
+		)
+		(pad "69" thru_hole circle
+			(at 1.68 -2.8)
+			(size 0.5 0.5)
+			(drill 0.3)
+			(layers "*.Cu")
+			(remove_unused_layers no)
+			(net "GND")
+			(pinfunction "VSS_69")
+			(pintype "passive")
+		)
+		(pad "69" thru_hole circle
+			(at 1.68 2.8 180)
+			(size 0.5 0.5)
+			(drill 0.3)
+			(layers "*.Cu")
+			(remove_unused_layers no)
+			(net "GND")
+			(pinfunction "VSS_69")
+			(pintype "passive")
+		)
+		(pad "69" thru_hole circle
+			(at 2.8 -2.8 270)
+			(size 0.5 0.5)
+			(drill 0.3)
+			(property pad_prop_heatsink)
+			(layers "*.Cu")
+			(remove_unused_layers no)
+			(net "GND")
+			(pinfunction "VSS_69")
+			(pintype "passive")
+		)
+		(pad "69" thru_hole circle
+			(at 2.8 -1.68 270)
+			(size 0.5 0.5)
+			(drill 0.3)
+			(layers "*.Cu")
+			(remove_unused_layers no)
+			(net "GND")
+			(pinfunction "VSS_69")
+			(pintype "passive")
+		)
+		(pad "69" thru_hole circle
+			(at 2.8 -0.56 270)
+			(size 0.5 0.5)
+			(drill 0.3)
+			(layers "*.Cu")
+			(remove_unused_layers no)
+			(net "GND")
+			(pinfunction "VSS_69")
+			(pintype "passive")
+		)
+		(pad "69" thru_hole circle
+			(at 2.8 0.56 270)
+			(size 0.5 0.5)
+			(drill 0.3)
+			(layers "*.Cu")
+			(remove_unused_layers no)
+			(net "GND")
+			(pinfunction "VSS_69")
+			(pintype "passive")
+		)
+		(pad "69" thru_hole circle
+			(at 2.8 1.68 270)
+			(size 0.5 0.5)
+			(drill 0.3)
+			(layers "*.Cu")
+			(remove_unused_layers no)
+			(net "GND")
+			(pinfunction "VSS_69")
+			(pintype "passive")
+		)
+		(pad "69" thru_hole circle
+			(at 2.8 2.8 180)
+			(size 0.5 0.5)
+			(drill 0.3)
+			(property pad_prop_heatsink)
+			(layers "*.Cu")
+			(remove_unused_layers no)
+			(net "GND")
+			(pinfunction "VSS_69")
+			(pintype "passive")
+		)
 		(embedded_fonts no)
