File: ali/v2/valvedrivers/valvedrivers.kicad_pcb (KiCad board)
At the start: 4 copper layers, 85 x 76 mm, 153 parts, among them J1 Conn_02x01, J10 Conn_01x02, J11 Conn_01x02, J12 Conn_01x02, J13 Conn_01x02, J14 Conn_01x02, J15 Conn_01x02, J16 Conn_01x02, J17 Conn_01x02, J18 Conn_01x02, J19 Conn_01x02, J2 Conn_01x05, J20 Conn_01x02, J21 Conn_01x02, J3 USB_C_Receptacle_USB2.0_16P, J4 Screw_Terminal_01x02, J5 Screw_Terminal_01x02, J6 Screw_Terminal_01x02, J7 Conn_01x05, J8 Conn_01x03, J9 Vertical Ethernet, SW1 SKRPANE010, U1 STM32H563RIV6, U10 PS2841-4B, U11 PS2841-4B, U12 IPS4140HQ, U13 PS2841-4B, U14 PS2841-4B, U2 LTV-816S, U3 AP2112K-3.3, U4 TJA1462ATK, U5 LAN8742AI, U6 IPS4140HQ, U7 PS2841-4B, U8 PS2841-4B, U9 IPS4140HQ, Y1 25 MHz, Y2 25 MHz

Commit message: Fix 50R/60R widths
Parts:
- moved R3 19.0 mm to (139.5, 75.7), turned to -90 degrees
- moved D1 16.6 mm to (141.7, 76.7), turned to 180 degrees
- moved J4 6.36 mm to (144.6, 69.8)
- moved F2 2.73 mm to (131.3, 80.5), turned to 90 degrees
- moved J7 0.90 mm to (163.4, 70.1)
Connections:
- net /Microcontroller/IGNIG_STAT renamed /Microcontroller/BRK_WIRE
- net /Microcontroller/PWR_STAT renamed /Microcontroller/+24V_STAT
- net Net-(J8-Pin_1) renamed /Connectivity/CAN+
- net Net-(J8-Pin_2) renamed /Connectivity/CAN-
Routing:
- net +24VCONN: track 13.6 -> 0.00 mm
- net /Drivers 2/MCU_IN1: track 25.1 -> 26.4 mm
- net /Drivers 2/MCU_IN2: track 25.1 -> 26.2 mm
- net +3.3V: track 92.9 -> 93.8 mm
- net /Microcontroller/IGNIG: track 54.9 -> 55.4 mm
- net GNDPWR: vias 228 -> 231
- net GND: vias 247 -> 252

Commit message: Begin prep for second board review
Parts:
- removed the C26 at (158.3, 119.8)
- removed D10, D11, D12, D13, D14, D15, D16, D17, D18, D19, D8, D9: SMF4L33CA, Diode_SMD:D_SOD-123F
- removed the D2 at (113.3, 77.5)
- removed the J9 at (168.3, 121.1)
- removed the R18 at (149.9, 119.4)
- removed the R20 at (169.5, 133.1)
- removed the R23 at (126.5, 94.3)
- removed the R4 at (113.3, 79.1)
- removed R48, R49, R50, R51, R54, R55, R56, R57: 10k, APRL_Passive:R_0603
- removed R52, R53: 1k, APRL_Passive:R_0603
- removed U12: IPS4140HQ, APRL_Package:QFN-48_EP_9.01x7.01_Pitch0.5mm
- removed U13, U14: PS2841-4B, APRL_Package:SOIC-12
- removed the U6 at (111.7, 85.3)
- added C24: 220nF, APRL_Passive:C_0603, B.Cu at (158.6, 119.8)
- added C32: 10nF, APRL_Passive:C_0603, B.Cu at (99.7, 76.5)
- added C33: 10nF, APRL_Passive:C_0603, B.Cu at (99.7, 83.8)
- added C34: 10nF, APRL_Passive:C_0603, B.Cu at (99.7, 90.8)
- added C35: 10nF, APRL_Passive:C_0603, B.Cu at (99.7, 97.9)
- added C36: 47uF, APRL_Passive:KEMET MU VIB, F.Cu at (118.6, 97.2)
- added C37: 100nF, APRL_Passive:C_0603, F.Cu at (112.6, 100.7)
- added C38: 10nF, APRL_Passive:C_0603, B.Cu at (99.7, 105.3)
- added C39: 10nF, APRL_Passive:C_0603, B.Cu at (99.7, 112.5)
- added C40: 10nF, APRL_Passive:C_0603, B.Cu at (99.7, 119.7)
- added C41: 10nF, APRL_Passive:C_0603, B.Cu at (99.7, 126.9)
- added C42: 47uF, APRL_Passive:KEMET MU VIB, F.Cu at (118.0, 120.2)
- added C43: 100nF, APRL_Passive:C_0603, F.Cu at (121.7, 126.4)
- added C44: 100nF, APRL_Passive:C_0603, F.Cu at (133.3, 118.5)
- added C45: 10nF, APRL_Passive:C_0603, B.Cu at (109.5, 135.8)
- added C46: 10nF, APRL_Passive:C_0603, B.Cu at (116.6, 135.8)
- added C47: 10nF, APRL_Passive:C_0603, B.Cu at (123.8, 135.8)
- added C48: 10nF, APRL_Passive:C_0603, B.Cu at (131.2, 135.8)
- added F4: 100mA, APRL_Passive:Fuse_0805_2012Metric, B.Cu at (172.0, 72.1)
- added J8: Vertical Ethernet, APRL_Connector:RJ45_Hanrun_HY951180A_Vertical, F.Cu at (168.3, 121.1)
- added R11: 10k, APRL_Passive:R_0603, F.Cu at (169.0, 96.8)
- added R12: 1k, APRL_Passive:R_0603, B.Cu at (175.7, 76.1)
- added R19: 12.1k, APRL_Passive:R_0603, F.Cu at (150.0, 119.4)
- added R9: 10k, APRL_Passive:R_0603, F.Cu at (144.9, 84.3)
- added U4: LTV-816S, APRL_Package:4-SMD, B.Cu at (175.7, 78.9)
- C30, C31: value 47uF -> 100nF; footprint APRL_Passive:KEMET MU VIB -> APRL_Passive:C_0603
- R1, R2: value 4.7k -> 5.1k
- R10, R36, R37, R38, R39, U2: moved to F.Cu
- R22: value 1k -> 330R; moved to F.Cu
- R28, R29, R34, R35, R40, R41, R46, R47: value 1k -> 10k
- R3: value 150k -> 100k
- R30, R31, R32, R33, R42, R43, R44, R45: moved to B.Cu
- U10, U7: value PS2841-4B -> SN74CBTLV3245A; footprint APRL_Package:SOIC-12 -> APRL_Package:TSSOP-20_4.4x6.5mm_P0.65mm; moved to F.Cu
- U11, U8: value PS2841-4B -> IPS4140HQ; footprint APRL_Package:SOIC-12 -> APRL_Package:QFN-48_EP_9.01x7.01_Pitch0.5mm
- moved R22 49.3 mm to (174.0, 109.9), turned to 90 degrees
- moved C29 41.2 mm to (124.1, 82.8), turned to 0 degrees
- moved J5 30.5 mm to (146.0, 69.7)
- moved J13 28.9 mm to (103.7, 98.7)
- moved J17 28.9 mm to (103.6, 127.6)
- moved J12 28.9 mm to (103.6, 91.5)
- moved J16 28.9 mm to (103.6, 120.4)
- moved J10 28.9 mm to (103.7, 77.1)
- moved J14 28.9 mm to (103.6, 106.0)
- moved J11 28.8 mm to (103.7, 84.4)
- moved J15 28.8 mm to (103.6, 113.2)
- moved J4 27.8 mm to (116.8, 69.7)
- moved D1 27.6 mm to (114.2, 78.5)
- moved R3 25.7 mm to (114.2, 80.3), turned to 180 degrees
- moved R21 23.6 mm to (169.5, 133.1), turned to -90 degrees
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- renumbered C23 to C22, C24 to C23, C27 to C25, C28 to C26, C22 to C27, C25 to C28, D3 to D2, D4 to D3, D5 to D4, D6 to D5, D7 to D6, J14 to J10, J15 to J11, J16 to J12, J17 to J13, J10 to J14, J11 to J15, J12 to J16, J13 to J17, J8 to J9, R12 to R13, R13 to R14, R14 to R15, R15 to R16, R16 to R17, R17 to R18, R19 to R20, R11 to R23, R5 to R4, R6 to R5, R7 to R6, R8 to R7, R9 to R8, U4 to U6
Connections:
- net /Connectivity/CAN+ renamed Net-(J9-Pin_1)
- net /Connectivity/CAN- renamed Net-(J9-Pin_2)
- net /Connectivity/LED2-INTSEL renamed Net-(U5-LED2/~{INTSEL})
- net /Connectivity/RX+ renamed Net-(J8-RD+)
- net /Connectivity/RX- renamed Net-(J8-RD-)
- net /Connectivity/TX+ renamed Net-(J8-TD+)
- net /Connectivity/TX- renamed Net-(J8-TD-)
- net /Microcontroller/USER_LED_1 renamed Net-(U1-PC6)
- net /Microcontroller/USER_LED_2 renamed Net-(U1-PC7)
- net /Microcontroller/USER_LED_3 renamed Net-(U1-PC8)
- C29 pad 2: GNDPWR -> GND
- C30 pad 2: GNDPWR -> GND
- C31 pad 1: +24V -> +3.3V
- C31 pad 2: GNDPWR -> GND
- D1 pad 1: GNDPWR -> GND
- F2 pad 1: +24VIN -> +24V
- F2 pad 2: +24VCONN -> Net-(J4-Pin_2)
- J10 pad 1: Net-(D12-A2) -> Net-(J10-Pin_1)
- J10 pad 2: GNDPWR -> GND
- J11 pad 1: Net-(D13-A2) -> Net-(J11-Pin_1)
- J11 pad 2: GNDPWR -> GND
- J12 pad 1: Net-(D14-A2) -> Net-(J12-Pin_1)
- J12 pad 2: GNDPWR -> GND
- J13 pad 1: Net-(D15-A2) -> Net-(J13-Pin_1)
- J13 pad 2: GNDPWR -> GND
- J14 pad 1: Net-(D8-A2) -> Net-(J14-Pin_1)
- J14 pad 2: GNDPWR -> GND
- J15 pad 1: Net-(D9-A2) -> Net-(J15-Pin_1)
- J15 pad 2: GNDPWR -> GND
- J16 pad 1: Net-(D10-A2) -> Net-(J16-Pin_1)
- J16 pad 2: GNDPWR -> GND
- J17 pad 1: Net-(D11-A2) -> Net-(J17-Pin_1)
- J17 pad 2: GNDPWR -> GND
- J18 pad 1: Net-(D16-A2) -> Net-(J18-Pin_1)
- J18 pad 2: GNDPWR -> GND
- J19 pad 1: Net-(D17-A2) -> Net-(J19-Pin_1)
- J19 pad 2: GNDPWR -> GND
- J20 pad 1: Net-(D18-A2) -> Net-(J20-Pin_1)
- J20 pad 2: GNDPWR -> GND
- J21 pad 1: Net-(D19-A2) -> Net-(J21-Pin_1)
- J21 pad 2: GNDPWR -> GND
- J4 pad 1: GNDPWR -> GND
- J4 pad 2: +24VCONN -> Net-(J4-Pin_2)
- J5 pad 1: +24V -> Net-(J5-Pin_1)
- J5 pad 2: +24VIN -> +24V
- J7 pad 1: +5V -> +3.3V
- J7 pad 2: GND -> /Microcontroller/IGNIG
- J7 pad 3: /Microcontroller/BRK_WIRE -> Net-(J7-Pin_3)
- J7 pad 4: /Microcontroller/IGNIG -> GND
- J7 pad 5: +3.3V -> +5V
- R10 pad 1: +24V -> Net-(J5-Pin_1)
- R22 pad 1: /Drivers 1/MCU_IN4 -> Net-(J8-Pad11)
- R22 pad 2: Net-(R22-Pad2) -> GND
- R24 pad 1: /Drivers 1/IN1 -> +3.3V
- R24 pad 2: GNDPWR -> /Driver Set 1/MCU_STAT1
- R25 pad 1: /Drivers 1/IN2 -> +3.3V
- R25 pad 2: GNDPWR -> /Driver Set 1/MCU_STAT2
- R26 pad 1: /Drivers 1/IN3 -> +3.3V
- R26 pad 2: GNDPWR -> /Driver Set 1/MCU_STAT3
- R27 pad 1: /Drivers 1/IN4 -> +3.3V
- R27 pad 2: GNDPWR -> /Driver Set 1/MCU_STAT4
- R28 pad 1: /Drivers 1/MCU_IN2 -> Net-(U7-B5)
- R28 pad 2: Net-(R28-Pad2) -> GND
- R29 pad 1: /Drivers 1/MCU_IN1 -> Net-(U7-B6)
- R29 pad 2: Net-(R29-Pad2) -> GND
- R3 pad 1: +24VCONN -> +24V
- R30 pad 1: Net-(R30-Pad1) -> Net-(U7-B7)
- R30 pad 2: /Drivers 1/STAT4 -> GND
- R31 pad 1: Net-(R31-Pad1) -> Net-(U7-B8)
- R31 pad 2: /Drivers 1/STAT3 -> GND
- R32 pad 1: Net-(R32-Pad1) -> +3.3V
- R32 pad 2: /Drivers 1/STAT2 -> /Driver Set 1/MCU_STAT5
- R33 pad 1: Net-(R33-Pad1) -> +3.3V
- R33 pad 2: /Drivers 1/STAT1 -> /Driver Set 1/MCU_STAT6
- R34 pad 1: /Drivers 2/MCU_IN4 -> +3.3V
- R34 pad 2: Net-(R34-Pad2) -> /Driver Set 1/MCU_STAT7
- R35 pad 1: /Drivers 2/MCU_IN3 -> +3.3V
- R35 pad 2: Net-(R35-Pad2) -> /Driver Set 1/MCU_STAT8
- R36 pad 1: /Drivers 2/IN1 -> Net-(U7-B1)
- R36 pad 2: GNDPWR -> GND
- R37 pad 1: /Drivers 2/IN2 -> Net-(U7-B2)
- R37 pad 2: GNDPWR -> GND
- R38 pad 1: /Drivers 2/IN3 -> Net-(U7-B3)
- R38 pad 2: GNDPWR -> GND
- R39 pad 1: /Drivers 2/IN4 -> Net-(U7-B4)
- R39 pad 2: GNDPWR -> GND
- R40 pad 1: /Drivers 2/MCU_IN2 -> +3.3V
- R40 pad 2: Net-(R40-Pad2) -> /Driver Set 2/MCU_STAT9
- R41 pad 1: /Drivers 2/MCU_IN1 -> +3.3V
- R41 pad 2: Net-(R41-Pad2) -> /Driver Set 2/MCU_STAT10
- R42 pad 1: Net-(R42-Pad1) -> +3.3V
- R42 pad 2: /Drivers 2/STAT4 -> /Driver Set 2/MCU_STAT11
- R43 pad 1: Net-(R43-Pad1) -> +3.3V
- R43 pad 2: /Drivers 2/STAT3 -> /Driver Set 2/MCU_STAT12
- R44 pad 1: Net-(R44-Pad1) -> Net-(U10-B1)
- R44 pad 2: /Drivers 2/STAT2 -> GND
- R45 pad 1: Net-(R45-Pad1) -> Net-(U10-B3)
- R45 pad 2: /Drivers 2/STAT1 -> GND
- R46 pad 1: /Drivers 3/MCU_IN4 -> Net-(U10-B5)
- R46 pad 2: Net-(R46-Pad2) -> GND
- R47 pad 1: /Drivers 3/MCU_IN3 -> Net-(U10-B7)
- R47 pad 2: Net-(R47-Pad2) -> GND
- U1 pad 10: unconnected-(U1-PC2-Pad10) -> /Driver Set 1/MCU_STAT6
- U1 pad 11: unconnected-(U1-PC3-Pad11) -> /Driver Set 1/MCU_STAT7
- U1 pad 17: /Drivers 1/MCU_IN4 -> /Driver Set 1/MCU_STAT8
- U1 pad 2: unconnected-(U1-PC13-Pad2) -> /Driver Set 1/MCU_STAT2
- U1 pad 20: /Drivers 1/MCU_IN3 -> /Driver Set 2/MCU_IN9
- U1 pad 21: /Drivers 1/MCU_IN2 -> /Driver Set 2/MCU_IN10
- U1 pad 22: /Drivers 1/MCU_IN1 -> /Driver Set 2/MCU_IN11
- U1 pad 26: /Drivers 2/MCU_IN4 -> /Driver Set 2/MCU_IN12
- U1 pad 27: /Drivers 2/MCU_IN3 -> /Driver Set 2/MCU_STAT9
- U1 pad 28: /Drivers 2/MCU_IN2 -> /Driver Set 2/MCU_STAT10
- U1 pad 29: /Drivers 2/MCU_IN1 -> /Driver Set 2/MCU_STAT11
- U1 pad 3: /Drivers 3/MCU_STAT3 -> /Driver Set 1/MCU_STAT3
- U1 pad 35: /Drivers 3/MCU_IN4 -> /Driver Set 2/MCU_STAT12
- U1 pad 36: /Drivers 3/MCU_IN3 -> unconnected-(U1-PB14-Pad36)
- U1 pad 38: /Drivers 3/MCU_IN2 -> unconnected-(U1-PD11-Pad38)
- U1 pad 39: /Drivers 3/MCU_IN1 -> unconnected-(U1-PD12-Pad39)
- U1 pad 4: /Drivers 3/MCU_STAT2 -> /Driver Set 1/MCU_STAT4
- U1 pad 44: /Microcontroller/BRK_WIRE -> /Microcontroller/~{BRK_STAT}
- U1 pad 45: /Microcontroller/+24V_STAT -> /Driver Set 1/~{BUSS_EN}
- U1 pad 55: /Drivers 1/MCU_STAT4 -> /Driver Set 1/MCU_IN1
- U1 pad 56: /Drivers 1/MCU_STAT3 -> /Driver Set 1/MCU_IN2
- U1 pad 57: /Drivers 1/MCU_STAT2 -> /Driver Set 1/MCU_IN3
- U1 pad 58: /Drivers 1/MCU_STAT1 -> /Driver Set 1/MCU_IN4
- U1 pad 59: /Drivers 2/MCU_STAT4 -> /Driver Set 1/MCU_IN5
- U1 pad 60: /Drivers 2/MCU_STAT3 -> /Driver Set 1/MCU_IN6
- U1 pad 61: /Drivers 2/MCU_STAT2 -> /Driver Set 1/MCU_IN7
- U1 pad 63: /Drivers 2/MCU_STAT1 -> /Driver Set 1/MCU_IN8
- U1 pad 64: /Drivers 3/MCU_STAT4 -> /Driver Set 1/MCU_STAT1
- U1 pad 8: /Drivers 3/MCU_STAT1 -> /Driver Set 1/MCU_STAT5
- U10 pad 1: GND -> unconnected-(U10-NC-Pad1)
- U10 pad 10: /Drivers 2/IN3 -> GND
- U10 pad 11: /Drivers 2/IN4 -> unconnected-(U10-B8-Pad11)
- U10 pad 12: +24V -> Net-(U10-B7)
- U10 pad 2: Net-(R34-Pad2) -> /Driver Set 2/MCU_IN12
- U10 pad 3: Net-(R35-Pad2) -> unconnected-(U10-A2-Pad3)
- U10 pad 4: Net-(R40-Pad2) -> /Driver Set 2/MCU_IN11
- U10 pad 5: Net-(R41-Pad2) -> unconnected-(U10-A4-Pad5)
- U10 pad 6: GND -> /Driver Set 2/MCU_IN10
- U10 pad 7: +24V -> unconnected-(U10-A6-Pad7)
- U10 pad 8: /Drivers 2/IN1 -> /Driver Set 2/MCU_IN9
- U10 pad 9: /Drivers 2/IN2 -> unconnected-(U10-A8-Pad9)
- U11 pad 1: +24V -> unconnected-(U11-NC-Pad1)
- U11 pad 10: /Drivers 2/MCU_STAT3 -> unconnected-(U11-NC-Pad10)
- U11 pad 11: /Drivers 2/MCU_STAT4 -> unconnected-(U11-NC-Pad11)
- U11 pad 12: +3.3V -> unconnected-(U11-NC-Pad12)
- U11 pad 2: Net-(R42-Pad1) -> unconnected-(U11-NC-Pad2)
- U11 pad 3: Net-(R43-Pad1) -> unconnected-(U11-NC-Pad3)
- U11 pad 4: Net-(R44-Pad1) -> unconnected-(U11-NC-Pad4)
- U11 pad 5: Net-(R45-Pad1) -> unconnected-(U11-NC-Pad5)
- U11 pad 6: +24V -> unconnected-(U11-NC-Pad6)
- U11 pad 7: +3.3V -> unconnected-(U11-NC-Pad7)
- U11 pad 8: /Drivers 2/MCU_STAT1 -> unconnected-(U11-NC-Pad8)
- U11 pad 9: /Drivers 2/MCU_STAT2 -> unconnected-(U11-NC-Pad9)
- U2 pad 2: GNDPWR -> GND
- U2 pad 3: /Microcontroller/+24V_STAT -> GND
- U2 pad 4: +3.3V -> /Driver Set 1/~{BUSS_EN}
- U5 pad 3: /Connectivity/LED1-REGOFF -> Net-(U5-LED1/REGOFF)
- U7 pad 1: GND -> unconnected-(U7-NC-Pad1)
- U7 pad 10: /Drivers 1/IN3 -> GND
- U7 pad 11: /Drivers 1/IN4 -> Net-(U7-B8)
- U7 pad 12: +24V -> Net-(U7-B7)
- U7 pad 2: Net-(R22-Pad2) -> /Driver Set 1/MCU_IN8
- U7 pad 3: Net-(R23-Pad2) -> /Driver Set 1/MCU_IN7
- U7 pad 4: Net-(R28-Pad2) -> /Driver Set 1/MCU_IN6
- U7 pad 5: Net-(R29-Pad2) -> /Driver Set 1/MCU_IN5
- U7 pad 6: GND -> /Driver Set 1/MCU_IN4
- U7 pad 7: +24V -> /Driver Set 1/MCU_IN3
- U7 pad 8: /Drivers 1/IN1 -> /Driver Set 1/MCU_IN2
- U7 pad 9: /Drivers 1/IN2 -> /Driver Set 1/MCU_IN1
- U8 pad 1: +24V -> unconnected-(U8-NC-Pad1)
- U8 pad 10: /Drivers 1/MCU_STAT3 -> unconnected-(U8-NC-Pad10)
- U8 pad 11: /Drivers 1/MCU_STAT4 -> unconnected-(U8-NC-Pad11)
- U8 pad 12: +3.3V -> unconnected-(U8-NC-Pad12)
- U8 pad 2: Net-(R30-Pad1) -> unconnected-(U8-NC-Pad2)
- U8 pad 3: Net-(R31-Pad1) -> unconnected-(U8-NC-Pad3)
- U8 pad 4: Net-(R32-Pad1) -> unconnected-(U8-NC-Pad4)
- U8 pad 5: Net-(R33-Pad1) -> unconnected-(U8-NC-Pad5)
- U8 pad 6: +24V -> unconnected-(U8-NC-Pad6)
- U8 pad 7: +3.3V -> unconnected-(U8-NC-Pad7)
- U8 pad 8: /Drivers 1/MCU_STAT1 -> unconnected-(U8-NC-Pad8)
- U8 pad 9: /Drivers 1/MCU_STAT2 -> unconnected-(U8-NC-Pad9)
- U9 pad 13: /Drivers 2/IN1 -> Net-(U7-B1)
- U9 pad 14: /Drivers 2/STAT1 -> /Driver Set 1/MCU_STAT8
- U9 pad 15: /Drivers 2/IN2 -> Net-(U7-B2)
- U9 pad 16: /Drivers 2/STAT2 -> /Driver Set 1/MCU_STAT7
- U9 pad 17: GNDPWR -> GND
- U9 pad 18: /Drivers 2/STAT3 -> /Driver Set 1/MCU_STAT6
- U9 pad 19: /Drivers 2/IN3 -> Net-(U7-B3)
- U9 pad 20: /Drivers 2/STAT4 -> /Driver Set 1/MCU_STAT5
- U9 pad 21: /Drivers 2/IN4 -> Net-(U7-B4)
- U9 pad 36: Net-(D12-A2) -> Net-(J14-Pin_1)
- U9 pad 37: Net-(D12-A2) -> Net-(J14-Pin_1)
- U9 pad 38: Net-(D12-A2) -> Net-(J14-Pin_1)
- U9 pad 39: Net-(D13-A2) -> Net-(J15-Pin_1)
- U9 pad 40: Net-(D13-A2) -> Net-(J15-Pin_1)
- U9 pad 41: Net-(D13-A2) -> Net-(J15-Pin_1)
- U9 pad 42: Net-(D14-A2) -> Net-(J16-Pin_1)
- U9 pad 43: Net-(D14-A2) -> Net-(J16-Pin_1)
- U9 pad 44: Net-(D14-A2) -> Net-(J16-Pin_1)
- U9 pad 45: Net-(D15-A2) -> Net-(J17-Pin_1)
- U9 pad 46: Net-(D15-A2) -> Net-(J17-Pin_1)
- U9 pad 47: Net-(D15-A2) -> Net-(J17-Pin_1)
Routing:
- net /Driver Set 1/~{BUSS_EN}: track 0.00 -> 86.9 mm, vias 0 -> 2
- net +24V: track 71.2 -> 0.00 mm, vias 40 -> 43
- net /Microcontroller/BRK_WIRE: track 53.3 -> 0.00 mm, vias 3 -> 0
- net Net-(U5-LED1/REGOFF): track 0.00 -> 44.9 mm
- net /Connectivity/LED1-REGOFF: track 44.9 -> 0.00 mm
- net /Microcontroller/+24V_STAT: track 43.9 -> 0.00 mm, vias 3 -> 0
- net /Microcontroller/~{BRK_STAT}: track 0.00 -> 38.7 mm, vias 0 -> 5
- net /Drivers 3/MCU_IN1: track 35.1 -> 0.00 mm, vias 1 -> 0
- net /Drivers 3/MCU_IN2: track 35.0 -> 0.00 mm, vias 1 -> 0
- net /Drivers 3/MCU_STAT4: track 34.9 -> 0.00 mm
- net /Driver Set 1/MCU_STAT1: track 0.00 -> 32.7 mm, vias 0 -> 2
- net /Drivers 3/MCU_STAT3: track 32.5 -> 0.00 mm
- net /Driver Set 2/MCU_STAT12: track 0.00 -> 32.5 mm, vias 0 -> 2
- net /Drivers 2/MCU_STAT4: track 32.4 -> 0.00 mm
- net /Drivers 3/MCU_IN3: track 32.1 -> 0.00 mm, vias 1 -> 0
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- added copper zone on F.Cu, net Net-(J10-Pin_1)
- added copper zone on F.Cu, net Net-(J11-Pin_1)
- added copper zone on F.Cu, net Net-(J12-Pin_1)
- added copper zone on F.Cu, net Net-(J13-Pin_1)
- added copper zone on F.Cu, net Net-(J14-Pin_1)
- added copper zone on F.Cu, net Net-(J15-Pin_1)
- added copper zone on F.Cu, net Net-(J16-Pin_1)
- added copper zone on F.Cu, net Net-(J17-Pin_1)
- added copper zone on F.Cu, net Net-(J18-Pin_1)
- added copper zone on F.Cu, net Net-(J19-Pin_1)
- added copper zone on F.Cu, net Net-(J20-Pin_1)
- added copper zone on F.Cu, net Net-(J21-Pin_1)
- added copper zone on F.Cu, net Net-(J4-Pin_2)
- removed copper zone on F.Cu, net +24VCONN
- removed copper zone on B.Cu, net +24VIN
- removed copper zone on B.Cu, net GNDPWR
- removed copper zone on F.Cu, net GNDPWR
- removed copper zone on In1.Cu, net GNDPWR
- removed copper zone on In2.Cu, net GNDPWR
- removed copper zone on F.Cu, net Net-(D10-A2)
- removed copper zone on F.Cu, net Net-(D11-A2)
- removed copper zone on F.Cu, net Net-(D12-A2)
- removed copper zone on F.Cu, net Net-(D13-A2)
- removed copper zone on F.Cu, net Net-(D14-A2)
- removed copper zone on F.Cu, net Net-(D15-A2)
- removed copper zone on F.Cu, net Net-(D16-A2)
- removed copper zone on F.Cu, net Net-(D17-A2)
- removed copper zone on F.Cu, net Net-(D18-A2)
- removed copper zone on F.Cu, net Net-(D19-A2)
- removed copper zone on F.Cu, net Net-(D8-A2)
- removed copper zone on F.Cu, net Net-(D9-A2)
Other:
- board text added: "10A"
- board text removed: "FUSE"
