File: ali/v2/valvedrivers/microcontroller.kicad_sch (KiCad schematic)
At the start: 49 parts, among them J1 Conn_02x01, J2 Conn_01x05, J3 USB_C_Receptacle_USB2.0_16P, J4 Screw_Terminal_01x02, J5 Screw_Terminal_01x02, J6 Screw_Terminal_01x02, J7 Conn_01x05, SW1 SKRPANE010, U1 STM32H563RIV6, U2 LTV-816S, U3 AP2112K-3.3, Y1 25 MHz

Commit message: Begin prep for second board review
Parts:
- removed D1, D7: LED, APRL_Passive:LED_0603, symbol Device:LED_Small
- removed R3: 150k, APRL_Passive:R_0603, symbol Device:R_Small_US
- added D5: LED, APRL_Passive:LED_0603, symbol Device:LED_Small
- added F4: 100mA, APRL_Passive:Fuse_0805_2012Metric, symbol Device:Fuse_Small
- added R11, R9: 10k, APRL_Passive:R_0603, symbol Device:R_Small_US
- added R12: 1k, APRL_Passive:R_0603, symbol Device:R_Small_US
- added U4: LTV-816S, APRL_Package:4-SMD, symbol Isolator:PC817
- R1, R2: value 4.7k -> 5.1k; MPN RC0603FR-074K7L -> RC0603FR-075K1L
- R3: renamed from R4; value 150k -> 100k; MPN RC0603FR-07150KL -> RC0603FR-07100KL
- U2: footprint Package_DIP:DIP-4_W7.62mm -> APRL_Package:4-SMD
- renumbered D2 to D1, D3 to D2, D4 to D3, D5 to D4, R5 to R4, R6 to R5, R7 to R6, R8 to R7, R9 to R8
Connections:
- net +24VIN is gone; now on net +24V: F2.1, J5.2 (Pin_2)
- net GNDPWR is gone; now on net GND: D1.1 (K), J4.1 (Pin_1), U2.2
- net +24V: no longer J5.1 (Pin_1), R10.1
- net +3.3V: now also J7.1 (Pin_1), R11.1, R9.1; no longer J7.5 (Pin_5), U2.4
- net +5V: now also J7.5 (Pin_5); no longer J7.1 (Pin_1)
- net GND: now also J7.4 (Pin_4), U2.3, D5.1 (K), U4.2, U4.3; no longer J7.2 (Pin_2)
- net IGNIG: now also J7.2 (Pin_2); no longer J7.4 (Pin_4)
- net IN_DRV1: now also U1.55 (PC11); no longer U1.22 (PA6)
- net IN_DRV10: now also U1.21 (PA5); no longer U1.38 (PD11)
- net IN_DRV11: now also U1.22 (PA6); no longer U1.36 (PB14)
- net IN_DRV12: now also U1.26 (PB0); no longer U1.35 (PB13)
- net IN_DRV2: now also U1.56 (PC12); no longer U1.21 (PA5)
- net IN_DRV3: now also U1.57 (PB3(JTDO); no longer U1.20 (PA4)
- net IN_DRV4: now also U1.58 (PB4(NJTRST)); no longer U1.17 (PA3)
- net IN_DRV5: now also U1.59 (PB5); no longer U1.29 (PB10)
- net IN_DRV6: now also U1.60 (PB6); no longer U1.28 (PB2)
- net IN_DRV7: now also U1.61 (PB7); no longer U1.27 (PB1)
- net IN_DRV8: now also U1.63 (PB8); no longer U1.26 (PB0)
- net IN_DRV9: now also U1.20 (PA4); no longer U1.39 (PD12)
- net STAT_DRV1: now also U1.64 (PB9); no longer U1.58 (PB4(NJTRST))
- net STAT_DRV10: now also U1.28 (PB2); no longer U1.4 (PC15)
- net STAT_DRV11: now also U1.29 (PB10); no longer U1.3 (PC14)
- net STAT_DRV12: now also U1.35 (PB13); no longer U1.64 (PB9)
- net STAT_DRV2: now also U1.2 (PC13); no longer U1.57 (PB3(JTDO)
- net STAT_DRV3: now also U1.3 (PC14); no longer U1.56 (PC12)
- net STAT_DRV4: now also U1.4 (PC15); no longer U1.55 (PC11)
- net STAT_DRV5: now also U1.8 (PC0); no longer U1.63 (PB8)
- net STAT_DRV6: now also U1.10 (PC2); no longer U1.61 (PB7)
- net STAT_DRV7: now also U1.11 (PC3); no longer U1.60 (PB6)
- net STAT_DRV8: now also U1.17 (PA3); no longer U1.59 (PB5)
- net STAT_DRV9: now also U1.27 (PB1); no longer U1.8 (PC0)
- net at D6.2 (A): now also R8.1; no longer R7.1
- net +24VCONN: no longer names the net of F2.2, J4.2 (Pin_2)
- net +24V_STAT renamed ~{BUSS_EN}
- net ~{BUSS_EN}: now also U2.4, R9.2; no longer U2.3
- net BRK_WIRE: no longer names the net of J7.3 (Pin_3)
- net BRK_WIRE: now also F4.1; no longer U1.44 (PA8)
- net USER_LED_1: no longer names the net of R6.2, U1.40 (PC6)
- net USER_LED_2: no longer names the net of R7.2, U1.41 (PC7)
- net USER_LED_3: no longer names the net of R8.2, U1.42 (PC8)
- new net: J5.1 (Pin_1), R10.1
- new net: F4.2, R12.1
- new net: R12.2, U4.1
- new net: D5.2 (A), R7.1
- new net ~{BRK_STAT}: R11.2, U1.44 (PA8), U4.4
Other:
- note added: "ISOLATED I/O"
- note removed: "BUS SWITCH EMULATION"
- note removed: "IGNIG"
- note removed: "Maybe consider adding a zener here to set a +24V UV threshold alert?"
- note removed: "The idea here is that a NC emergency stop button will be used to toggle the optocouplers driving the inputs of the drivers. When this line is cut, the pulldowns on the driver side take over, and the system pulls all outputs low, closing all solenoids."
- moved on the sheet: C12, C13, C14, C15, C16, C17, D1, D2, D3, D4, F1, F2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
Changed lines of the file:
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@@
 	(paper "USLetter")
 	(title_block
-		(date "2026-09-11")
+		(date "2026-10-10")
 	)
