File: ali/v2/valvedrivers/valvedrivers.kicad_sch (KiCad schematic)
At the start: 4 parts

Commit message: Begin prep for second board review
Other:
- sheet Drivers 1 renamed Driver Set 1
- removed sheet Drivers 2
- removed sheet Drivers 3
- added sheet Driver Set 2 (drivers2.kicad_sch)
- sheet Driver Set 1 ports: added MCU_IN5, MCU_IN6, MCU_IN7, MCU_IN8, MCU_STAT5, MCU_STAT6, MCU_STAT7, MCU_STAT8, ~{BUSS_EN}; removed none
- sheet Microcontroller ports: added ~{BUSS_EN}; removed none
