File: ali/v2/template/ali-template.kicad_pcb (KiCad board)
At the start: 4 copper layers, 76 x 76 mm, 71 parts, among them J1 Conn_02x01, J2 Conn_01x05, J3 USB_C_Receptacle_USB2.0_16P, J6 Screw_Terminal_01x02, J7 Conn_01x03, J8 Vertical Ethernet, SW1 SKRPANE010, U1 STM32H563RIV6, U2 AP2112K-3.3, U3 TJA1462ATK, U4 LAN8742AI, Y1 25 MHz, Y2 25 MHz

Commit message: mfw pts
Parts:
- U3: footprint Package_SON:HVSON-8-1EP_3x3mm_P0.65mm_EP1.6x2.4mm -> APRL_Package_QFN:HVSON-8-1EP_3x3mm_P0.65mm_EP1.6x2.4mm_ThermalVias
- U4: footprint Package_DFN_QFN:VQFN-24-1EP_4x4mm_P0.5mm_EP2.5x2.5mm_ThermalVias -> APRL_Package_QFN:VQFN-24-1EP_4x4mm_P0.5mm_EP2.5x2.5mm_ThermalVias

Commit message: mfw LCs
Parts:
- moved H2 9.00 mm to (91.7, 68.3)
- moved H4 9.00 mm to (91.7, 134.3)
Routing:
- net /Microcontroller/~{RST}: track 61.1 -> 61.7 mm
- net GND: vias 258 -> 265
Other:
- board size 76 x 76 mm -> 85 x 76 mm
