File: ali/v2/loadcells/load-cell.kicad_pcb (KiCad board)
At the start: 4 copper layers, 85 x 76 mm, 140 parts, among them J1 Conn_02x01, J10 Conn_01x04, J11 Conn_01x04, J12 Conn_01x04, J2 Conn_01x05, J3 USB_C_Receptacle_USB2.0_16P, J4 Conn_01x15, J5 Conn_02x09_Counter_Clockwise, J6 Screw_Terminal_01x02, J7 Conn_01x03, J8 Vertical Ethernet, J9 Conn_01x04, SW1 SKRPANE010, U1 STM32H563RIV6, U2 AP2112K-3.3, U3 TJA1462ATK, U4 LAN8742AI, U5 ADS1261, U6 ADS1261, U7 ADS1261, U8 ADS1261, Y1 25 MHz, Y2 7.3278 MHz, Y3 25 MHz

Commit message: Globally remove LCSC labels, update MPNs and IOCs, add +5V monitoring to DAQs, fix some footprints
Parts:
- added R27: 10k, APRL_Passive:R_0603, F.Cu at (157.4, 105.3)
- added R29: 10k, APRL_Passive:R_0603, F.Cu at (155.8, 104.8)
- Y2: value 7.3278 MHz -> 7.3728 MHz
Connections:
- J5 pad 11: /Microcontroller/PA6 -> /Microcontroller/PB0
- J5 pad 13: /Microcontroller/PB0 -> /Microcontroller/PA6
- U1 pad 27: unconnected-(U1-PB1-Pad27) -> /Microcontroller/+5V_SENSE
Routing:
- net /Microcontroller/+5V_SENSE: track 0.00 -> 19.8 mm, vias 0 -> 2
- net /Microcontroller/PB0: track 42.2 -> 39.5 mm, vias 2 -> 1
- net GND: track 2.94 -> 5.53 mm, vias 383 -> 385
- net +5V: track 24.7 -> 27.1 mm, vias 28 -> 29
- net /Microcontroller/PB2: track 37.7 -> 39.0 mm
- net /Microcontroller/PD11: track 48.7 -> 49.8 mm
- net /Microcontroller/PA6: track 38.6 -> 39.7 mm
- net Net-(U8-AIN7): track 7.00 -> 6.46 mm
- net Net-(U6-AIN7): track 7.00 -> 6.46 mm
- net Net-(U5-AIN7): track 7.00 -> 6.46 mm
- net Net-(U7-AIN7): track 7.00 -> 6.46 mm

Commit message: Re-link loadcell reference designators
Parts:
- renumbered D3 to D1, D4 to D2, D1 to D3, D2 to D4, R28 to R10, R8 to R11, R9 to R12, R10 to R13, R11 to R14, R12 to R15, R13 to R16, R14 to R17, R15 to R18, R16 to R19, R17 to R20, R18 to R21, R19 to R22, R20 to R23, R21 to R24, R22 to R25, R23 to R26, R24 to R27, R25 to R28, R26 to R29, R4 to R3, R5 to R4, R3 to R5, R27 to R7, R7 to R8, R29 to R9

Commit message: The other half of the great 10.0.6 migration
Routing:
- net GND: vias 385 -> 389
