File: ali/v2/loadcells/load-cell.kicad_pcb (KiCad board)
At the start: 4 copper layers, 85 x 76 mm, 142 parts, among them J1 Conn_02x01, J10 Conn_01x04, J11 Conn_01x04, J12 Conn_01x04, J2 Conn_01x05, J3 USB_C_Receptacle_USB2.0_16P, J4 Conn_01x15, J5 Conn_02x09_Counter_Clockwise, J6 Screw_Terminal_01x02, J7 Conn_01x03, J8 Vertical Ethernet, J9 Conn_01x04, SW1 SKRPANE010, U1 STM32H563RIV6, U2 AP2112K-3.3, U3 TJA1462ATK, U4 LAN8742AI, U5 ADS1261, U6 ADS1261, U7 ADS1261, U8 ADS1261, Y1 25 MHz, Y2 7.3728 MHz, Y3 25 MHz

Commit message: Fix 50R/60R widths
Connections:
- net Net-(J7-Pin_1) renamed /Connectivity/CAN+
- net Net-(J7-Pin_2) renamed /Connectivity/CAN-
Routing:
- net /Microcontroller/UART4_TX: track 24.5 -> 25.2 mm
- net /Microcontroller/UART4_RX: track 26.0 -> 26.7 mm
- net GND: vias 389 -> 390
- net (no net): vias 1 -> 0

Commit message: Begin prep for second board review
Parts:
- removed C12, C20, C31, C32, C51, C52: 100nF, APRL_Passive:C_0603
- removed the C23 at (159.6, 104.3)
- removed the C26 at (163.1, 105.8)
- removed C30, C33, C50, C53, C58, C68: 1uF, APRL_Passive:C_0603
- removed the C37 at (113.5, 83.9)
- removed the C38 at (119.3, 77.1)
- removed the C39 at (116.7, 83.9)
- removed the C40 at (116.3, 96.1)
- removed the C42 at (116.3, 90.7)
- removed the C43 at (114.7, 90.7)
- removed the C47 at (113.5, 97.8)
- removed C49, C59, C69: 10uF, APRL_Passive:C_0603
- removed C57, C67: 4.7nF, APRL_Passive:C_0603
- removed R10: 22R, APRL_Passive:R_0603
- removed R7, R9: 10k, APRL_Passive:R_0603
- removed U5, U8: ADS1261, APRL_Package_QFN:Texas_RHB0032E_VQFN-32-1EP_5x5mm_P0.5mm_EP3.45x3.45mm_ThermalVias
- removed the U7 at (115.1, 107.2)
- removed the Y2 at (122.9, 70.1)
- added C24: 100nF, APRL_Passive:C_0603, B.Cu at (147.8, 119.4)
- added C29: 100nF, APRL_Passive:C_0603, B.Cu at (163.0, 105.9)
- added C64: 1uF, APRL_Passive:C_0603, B.Cu at (121.3, 77.5)
- added R30: 1k, APRL_Passive:R_0603, F.Cu at (117.3, 82.9)
- C48: value 1uF -> 10nF
- D10, D11, D12, D13, D6, D7, D8, D9: value SMF7V0A -> VTVS28ASMF
- R1, R2: value 4.7k -> 5.1k
- R22, R23, R24, R25, R26, R27, R28, R29: value 1k -> 4.7k
- U6: value ADS1261 -> ADS124S08; footprint APRL_Package_QFN:Texas_RHB0032E_VQFN-32-1EP_5x5mm_P0.5mm_EP3.45x3.45mm_ThermalVias -> APRL_Package_QFN:Texas_RHB0032M_VQFN-32-1EP_5x5mm_P0.5mm_EP2.1x2.1mm_ThermalVias
- moved C60 45.4 mm to (124.1, 79.1), turned to 180 degrees
- moved C41 44.6 mm to (158.6, 104.0)
- moved C61 44.1 mm to (124.1, 80.7), turned to 180 degrees
- moved C63 39.4 mm to (119.6, 79.3), turned to 0 degrees
- moved C62 37.6 mm to (119.6, 80.9), turned to 0 degrees
- moved U6 13.1 mm to (121.9, 82.2)
- moved C48 6.76 mm to (117.3, 84.5), turned to 0 degrees
- moved C23 0.54 mm to (144.0, 120.8)
- moved C11 0.10 mm to (142.5, 93.4)
- moved R17 0.10 mm to (142.4, 123.0)
- renumbered C19 to C21, C21 to C23, C24 to C25, C25 to C26, C28 to C27, C29 to C28, C44 to C37, C46 to C38, C45 to C39, C27 to C40, C54 to C42, C56 to C43, C55 to C44, C64 to C45, C66 to C46, C65 to C47, J8 to J26, J7 to J8, R19 to R51, R20 to R52, R21 to R53, U3 to U4, U4 to U7, Y3 to Y2
Connections:
- net /ADC 1/SCLK renamed /ADC/SCLK
- net /Connectivity/CAN+ renamed Net-(J8-Pin_1)
- net /Connectivity/CAN- renamed Net-(J8-Pin_2)
- net /Connectivity/LED1-REGOFF renamed Net-(U7-LED1/REGOFF)
- net /Connectivity/LED2-INTSEL renamed Net-(U7-LED2/~{INTSEL})
- net /Connectivity/RX+ renamed Net-(J26-RD+)
- net /Connectivity/RX- renamed Net-(J26-RD-)
- net /Connectivity/TX+ renamed Net-(J26-TD+)
- net /Connectivity/TX- renamed Net-(J26-TD-)
- C34 pad 1: Net-(U5-AIN6) -> Net-(U6-GPIO0/AIN8)
- C35 pad 1: Net-(U5-AIN7) -> Net-(U6-GPIO1/AIN9)
- C35 pad 2: Net-(U5-AIN6) -> Net-(U6-GPIO0/AIN8)
- C36 pad 2: Net-(U5-AIN7) -> Net-(U6-GPIO1/AIN9)
- C37 pad 1: Net-(U6-AIN6) -> Net-(U6-AIN4)
- C38 pad 2: Net-(U6-AIN7) -> Net-(U6-AIN5)
- C39 pad 1: Net-(U6-AIN7) -> Net-(U6-AIN5)
- C39 pad 2: Net-(U6-AIN6) -> Net-(U6-AIN4)
- C42 pad 1: Net-(U7-AIN6) -> Net-(U6-AIN2)
- C43 pad 2: Net-(U7-AIN7) -> Net-(U6-AIN3)
- C44 pad 1: Net-(U7-AIN7) -> Net-(U6-AIN3)
- C44 pad 2: Net-(U7-AIN6) -> Net-(U6-AIN2)
- C45 pad 1: Net-(U8-AIN6) -> Net-(U6-AIN0)
- C46 pad 2: Net-(U8-AIN7) -> Net-(U6-AIN1)
- C47 pad 1: Net-(U8-AIN7) -> Net-(U6-AIN1)
- C47 pad 2: Net-(U8-AIN6) -> Net-(U6-AIN0)
- C48 pad 1: Net-(U6-BYPASS) -> GND
- C48 pad 2: GND -> Net-(U6-REFP0)
- C60 pad 1: +5V -> +3.3V
- C61 pad 1: +5V -> +3.3V
- C62 pad 1: +3.3V -> +5V
- C63 pad 1: +3.3V -> +5V
- J4 pad 10: /ADC 1/MISO -> /ADC/MISO
- J4 pad 11: /ADC 1/MOSI -> /ADC/MOSI
- J4 pad 3: /ADC 1/START -> /ADC/START
- J4 pad 4: /ADC 1/RESET -> /ADC/RESET
- R22 pad 2: Net-(U5-AIN6) -> Net-(U6-GPIO0/AIN8)
- R23 pad 2: Net-(U5-AIN7) -> Net-(U6-GPIO1/AIN9)
- R24 pad 2: Net-(U6-AIN6) -> Net-(U6-AIN4)
- R25 pad 2: Net-(U6-AIN7) -> Net-(U6-AIN5)
- R26 pad 2: Net-(U7-AIN6) -> Net-(U6-AIN2)
- R27 pad 2: Net-(U7-AIN7) -> Net-(U6-AIN3)
- R28 pad 2: Net-(U8-AIN6) -> Net-(U6-AIN0)
- R29 pad 2: Net-(U8-AIN7) -> Net-(U6-AIN1)
- U1 pad 10: /ADC 3/CS -> unconnected-(U1-PC2-Pad10)
- U1 pad 11: /ADC 4/CS -> unconnected-(U1-PC3-Pad11)
- U1 pad 2: /ADC 1/CS -> /ADC/CS
- U1 pad 27: /Microcontroller/+5V_SENSE -> unconnected-(U1-PB1-Pad27)
- U1 pad 3: /ADC 1/START -> /ADC/START
- U1 pad 4: /ADC 1/RESET -> /ADC/RESET
- U1 pad 57: /ADC 1/DRDY -> /ADC/DRDY
- U1 pad 58: /ADC 1/MISO -> /ADC/MISO
- U1 pad 59: /ADC 1/MOSI -> /ADC/MOSI
- U1 pad 8: /ADC 2/CS -> unconnected-(U1-PC0-Pad8)
- U6 pad 10: /ADC 2/CS -> /ADC/MOSI
- U6 pad 12: /ADC 1/MOSI -> /ADC/MISO
- U6 pad 13: /ADC 2/DRDY -> /ADC/DRDY
- U6 pad 14: /ADC 1/MISO -> GND
- U6 pad 15: Net-(U6-BYPASS) -> +3.3V
- U6 pad 16: GND -> +3.3V
- U6 pad 17: +3.3V -> GND
- U6 pad 18: /ADC 1/CLK -> /ADC/RESET
- U6 pad 2: Net-(U6-CAPP) -> Net-(U6-AIN5)
- U6 pad 21: unconnected-(U6-NC-Pad21) -> Net-(U6-GPIO1/AIN9)
- U6 pad 22: unconnected-(U6-NC-Pad22) -> Net-(U6-GPIO0/AIN8)
- U6 pad 23: unconnected-(U6-AIN9-Pad23) -> Net-(U6-REFOUT)
- U6 pad 24: unconnected-(U6-AIN8-Pad24) -> GND
- U6 pad 25: Net-(U6-AIN7) -> unconnected-(U6-NC-Pad25)
- U6 pad 26: Net-(U6-AIN6) -> +5V
- U6 pad 27: unconnected-(U6-AIN5/ACX2-Pad27) -> GND
- U6 pad 28: unconnected-(U6-AIN4/ACX1-Pad28) -> GND
- U6 pad 29: unconnected-(U6-AIN3/~{ACX2}-Pad29) -> GND
- U6 pad 3: Net-(U6-CAPN) -> Net-(U6-AIN4)
- U6 pad 30: unconnected-(U6-AIN2/~{ACX1}-Pad30) -> Net-(U6-REFP0)
- U6 pad 31: GND -> unconnected-(U6-REFN1/AIN7-Pad31)
- U6 pad 32: +5V -> unconnected-(U6-REFP1/AIN6-Pad32)
- U6 pad 4: +5V -> Net-(U6-AIN3)
- U6 pad 5: GND -> Net-(U6-AIN2)
- U6 pad 6: Net-(U6-REFOUT) -> Net-(U6-AIN1)
- U6 pad 7: +3.3V -> Net-(U6-AIN0)
- U6 pad 8: /ADC 1/RESET -> /ADC/START
- U6 pad 9: /ADC 1/START -> /ADC/CS
Routing:
- net /ADC 1/RESET: track 124.0 -> 0.00 mm, vias 4 -> 0
- net /ADC 1/MOSI: track 121.2 -> 0.00 mm, vias 6 -> 0
- net /ADC 1/MISO: track 117.3 -> 0.00 mm, vias 4 -> 0
- net /ADC 1/START: track 113.7 -> 0.00 mm, vias 4 -> 0
- net /ADC/SCLK: track 141.8 -> 67.0 mm, vias 6 -> 2
- net /ADC 1/CLK: track 71.1 -> 0.00 mm, vias 4 -> 0
- net /ADC/RESET: track 0.00 -> 57.4 mm, vias 0 -> 1
- net Net-(U6-AIN0): track 0.00 -> 50.2 mm
- net Net-(U6-AIN1): track 0.00 -> 48.4 mm
- net /ADC/MOSI: track 0.00 -> 47.6 mm, vias 0 -> 2
- net /ADC/MISO: track 0.00 -> 46.5 mm
- net /ADC 4/CS: track 41.9 -> 0.00 mm, vias 2 -> 0
- net /ADC/START: track 0.00 -> 39.7 mm, vias 0 -> 1
- net /ADC 1/DRDY: track 38.9 -> 0.00 mm, vias 2 -> 0
- net Net-(U6-AIN2): track 0.00 -> 35.5 mm
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- added copper zone on F.Cu, net Net-(U6-REFP0)
