File: ali/v2/loadcells/connectivity.kicad_sch (KiCad schematic)
At the start: 27 parts, among them J7 Conn_01x03, J8 Vertical Ethernet, U3 TJA1462ATK, U4 LAN8742AI, Y2 25 MHz

Commit message: mfw tcs
Parts:
- U3: footprint Package_SON:HVSON-8-1EP_3x3mm_P0.65mm_EP1.6x2.4mm -> APRL_Package_QFN:HVSON-8-1EP_3x3mm_P0.65mm_EP1.6x2.4mm_ThermalVias
- U4: footprint Package_DFN_QFN:VQFN-24-1EP_4x4mm_P0.5mm_EP2.5x2.5mm_ThermalVias -> APRL_Package_QFN:VQFN-24-1EP_4x4mm_P0.5mm_EP2.5x2.5mm_ThermalVias
Changed lines of the file:
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@@
 			)
 		)
-		(property "Footprint" "Package_DFN_QFN:VQFN-24-1EP_4x4mm_P0.5mm_EP2.5x2.5mm_ThermalVias"
+		(property "Footprint" "APRL_Package_QFN:VQFN-24-1EP_4x4mm_P0.5mm_EP2.5x2.5mm_ThermalVias"
 			(at 80.01 114.3 0)
 			(hide yes)
@@
 			)
 		)
-		(property "Footprint" "Package_SON:HVSON-8-1EP_3x3mm_P0.65mm_EP1.6x2.4mm"
+		(property "Footprint" "APRL_Package_QFN:HVSON-8-1EP_3x3mm_P0.65mm_EP1.6x2.4mm_ThermalVias"
 			(at 190.5 77.47 0)
 			(hide yes)

Commit message: Swap to sync'd ADS1261s on LC, update README and clean up Just scripts, some frame changes too.
Parts:
- renumbered C18 to C19, C19 to C20, C20 to C21, C21 to C22, C22 to C23, C23 to C24, C24 to C25, C25 to C26, C26 to C27, C27 to C28, C28 to C29, Y2 to Y3

Commit message: Globally remove LCSC labels, update MPNs and IOCs, add +5V monitoring to DAQs, fix some footprints
Parts:
- C25: MPN GRM21A5C2J471FWA1 -> GRM1885C1H471JA01
- C27: MPN GRM21AR72A224KAC5 -> GRM188R71H224KAC4
- renumbered R8 to R11, R9 to R12, R10 to R13, R11 to R14, R12 to R15, R13 to R16, R14 to R17, R15 to R18, R16 to R19, R17 to R20, R18 to R21

Commit message: Fix 50R/60R widths
Connections:
- net CAN+: now reaches J7.1 (Pin_1), R11.2, U3.7 (CANH)
- net CAN-: now reaches J7.2 (Pin_2), R11.1, U3.6 (CANL)
Changed lines of the file:
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@@
+		)
+	)
+	(label "CAN-"
+		(at 205.7332 67.31 0)
+		(effects
+			(font
+				(size 1.27 1.27)
+			)
+			(justify left bottom)
+		)
+	)
+	(label "CAN+"
+		(at 205.74 62.23 0)
+		(effects
+			(font
+				(size 1.27 1.27)
+			)
+			(justify left bottom)
 		)
 	)

Commit message: Begin prep for second board review
Parts:
- removed C19: 1uF, APRL_Passive:C_0603, symbol Device:C_Small
- removed C20: 100nF, APRL_Passive:C_0603, symbol Device:C_Small
- removed J7: Conn_01x03, APRL_Connector_Molex:Molex_CLIK-Mate_503159-0301_1x03-1MP_P1.50mm_Vertical, symbol Connector_Generic:Conn_01x03
- removed J8: Vertical Ethernet, APRL_Connector:RJ45_Hanrun_HY951180A_Vertical, symbol APRL_Connector:RJ45_Hanrun_HY951180A
- removed R19: 10k, APRL_Passive:R_0603, symbol Device:R_Small_US
- removed R20, R21: 330R, APRL_Passive:R_0603, symbol Device:R_Small_US
- removed U3: TJA1462ATK, APRL_Package_QFN:HVSON-8-1EP_3x3mm_P0.65mm_EP1.6x2.4mm_ThermalVias, symbol APRL_Comms:TJA1462ATK
- removed U4: LAN8742AI, APRL_Package_QFN:VQFN-24-1EP_4x4mm_P0.5mm_EP2.5x2.5mm_ThermalVias, symbol APRL_Comms:LAN8742A
- removed Y3: 25 MHz, APRL_Passive:3225-4P-L, symbol Device:Crystal_GND24
- added C40: 220nF, APRL_Passive:C_0603, symbol Device:C_Small
- added C41: 100nF, APRL_Passive:C_0603, symbol Device:C_Small
- added J26: Vertical Ethernet, APRL_Connector:RJ45_Hanrun_HY951180A_Vertical, symbol APRL_Connector:RJ45_Hanrun_HY951180A
- added J8: Conn_01x03, APRL_Connector_Molex:Molex_CLIK-Mate_503159-0301_1x03-1MP_P1.50mm_Vertical, symbol Connector_Generic:Conn_01x03
- added R51: 10k, APRL_Passive:R_0603, symbol Device:R_Small_US
- added R52, R53: 330R, APRL_Passive:R_0603, symbol Device:R_Small_US
- added U4: TJA1462ATK, APRL_Package_QFN:HVSON-8-1EP_3x3mm_P0.65mm_EP1.6x2.4mm_ThermalVias, symbol APRL_Comms:TJA1462ATK
- added U7: LAN8742AI, APRL_Package_QFN:VQFN-24-1EP_4x4mm_P0.5mm_EP2.5x2.5mm_ThermalVias, symbol APRL_Comms:LAN8742A
- added Y2: 25 MHz, APRL_Passive:3225-4P-L, symbol Device:Crystal_GND24
- C21: value 100nF -> 1uF; MPN GRM188R72A104KA35 -> GRM188D72A105KE01
- C24: value 1uF -> 100nF; MPN GRM188D72A105KE01 -> GRM188R72A104KA35
- C25: value 470pF -> 1uF; MPN GRM1885C1H471JA01 -> GRM188D72A105KE01
- C26: value 100nF -> 470pF; MPN GRM188R72A104KA35 -> GRM1885C1H471JA01
- C27: value 220nF -> 15pF; MPN GRM188R71H224KAC4 -> GRM1885C2E150FW07
- C29: value 15pF -> 100nF; MPN GRM1885C2E150FW07 -> GRM188R72A104KA35
Connections:
- net +3.3V: now also C23.1, C24.1, C29.1, C40.1, J26.3 (TCT), J26.5 (RCT), U4.5 (VIO), U7.1 (VDD2A), U7.19 (VDD1A), U7.9 (VDDIO); no longer C26.1, C27.1
- net +5V: now also C41.1, U4.3 (VCC); no longer C23.1
- net ETH_CRS_DV: now also U7.11 (CRS_DV/MODE2)
- net ETH_MDC: now also U7.13 (MDC)
- net ETH_MDIO: now also U7.12 (MDIO)
- net ETH_REF_CLK: now also U7.14 (~{INT}/REFCLKO)
- net ETH_RXD0: now also U7.8 (RXD0/MODE0)
- net ETH_RXD1: now also U7.7 (RXD1/MODE1)
- net ETH_TXD0: now also U7.17 (TXD0)
- net ETH_TXD1: now also U7.18 (TXD1)
- net ETH_TX_EN: now also U7.16 (TXEN)
- net ETH_~{RST}: now also U7.15 (~{RST})
- net FDCAN_RX: now also U4.4 (RXD)
- net FDCAN_STDBY: now also U4.8 (STB)
- net FDCAN_TX: now also U4.1 (TXD)
- net GND: now also C40.2, C41.2, J26.13, J26.14, J26.8, J8.3 (Pin_3), R51.2, R52.2, R53.2, U4.2 (GND), U4.9 (GND), U7.25 (VSS), Y2.2 (G), Y2.4 (G)
- net at C28.1: now also U7.4 (XTAL2), Y2.3
- net at C25.1: now also C26.1, U7.6 (VDDCR); no longer C24.1
- net at R17.2: now also U7.10 (RXER/PHYAD0)
- net at R18.1: now also U7.24 (RBIAS)
- net CAN+: no longer names the net of R11.2
- net CAN+: now also J8.1 (Pin_1), U4.7 (CANH)
- net CAN-: no longer names the net of R11.1
- net CAN-: now also J8.2 (Pin_2), U4.6 (CANL)
- net RX+: no longer names the net of R15.2
- net RX+: now also J26.6 (RD+), U7.23 (RXP)
- net RX-: no longer names the net of R16.2
- net RX-: now also J26.7 (RD-), U7.22 (RXN)
- net TX+: no longer names the net of R13.2
- net TX+: now also J26.1 (TD+), U7.21 (TXP)
- net TX-: no longer names the net of R14.2
- net TX-: now also J26.2 (TD-), U7.20 (TXN)
- new net: C27.1, U7.5 (XTAL1/CLKIN), Y2.1
- new net: J26.10, R52.1
- new net: J26.12, R51.1, U7.2 (LED2/~{INTSEL})
- new net: J26.9, U7.3 (LED1/REGOFF)
- new net: J26.11, R53.1
Other:
- note added: "ETH"
- note removed: "ETH JACK"
- note removed: "ETH PHY"
