File: ali/v2/loadcells/microcontroller.kicad_sch (KiCad schematic)
At the start: 46 parts, among them J1 Conn_02x01, J2 Conn_01x05, J3 USB_C_Receptacle_USB2.0_16P, J4 Conn_01x15, J5 Conn_02x09_Counter_Clockwise, J6 Screw_Terminal_01x02, SW1 SKRPANE010, U1 STM32H563RIV6, U2 AP2112K-3.3, Y1 25 MHz, Y2 7.3728 MHz

Commit message: Begin prep for second board review
Parts:
- removed C12: 100nF, APRL_Passive:C_0603, symbol Device:C_Small
- removed R10: 22R, APRL_Passive:R_0603, symbol Device:R_Small_US
- removed R7, R9: 10k, APRL_Passive:R_0603, symbol Device:R_Small_US
- removed Y2: 7.3728 MHz, APRL_Passive:Oscillator_SCTF_SX3M_3.2x2.5mm, symbol APRL_Misc:SX3M-xxxMHz
- R1, R2: value 4.7k -> 5.1k; MPN RC0603FR-074K7L -> RC0603FR-075K1L
Connections:
- net +5V_SENSE: no longer names the net of U1.27 (PB1)
- net ADC1_CS renamed ADC_CS
- net ADC2_CS: no longer names the net of U1.8 (PC0)
- net ADC3_CS: no longer names the net of U1.10 (PC2)
- net ADC4_CS: no longer names the net of U1.11 (PC3)
- no-connect marks 13 -> 14
Other:
- note removed: "ADC OSC"
- note removed: "Smaller CMOS crystals have undefined minimum rise times, so we're placing a series termination resistor just in case"
- note removed: "This spare GPIO header is not standardized, its literally just whatever I had available just so that we'd have it available if we ever needed it"
Changed lines of the file:
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@@
 	(paper "USLetter")
 	(title_block
-		(date "2026-09-11")
+		(date "2026-10-10")
 	)
