File: ali/v1/ThermoBoard/ThermoBoard.kicad_sch (KiCad schematic)
At the start: 4 parts

Commit message: Document setup, update template, and use an ampersand when referring to APRL
Other:
- company: Aggie Propulsion and Rocketry Lab -> Aggie Propulsion & Rocketry Lab
Changed lines of the file:
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@@
 		(date "2025-10-15")
 		(rev "1A")
-		(company "Aggie Propulsion and Rocketry Lab")
+		(company "Aggie Propulsion & Rocketry Lab")
 		(comment 1 "Drawn by: Nolan Poe")
 		(comment 2 "Checked by: Daniel Fan")
