File: ali/v1/ThermoBoard/can.kicad_sch (KiCad schematic)
At the start: 7 parts, among them J400 Conn_01x03, U400 TJA1042T-3

Commit message: Globally remove LCSC labels, update MPNs and IOCs, add +5V monitoring to DAQs, fix some footprints
Parts:
- C400, C401: LCSC C1525 -> (none)
- J400, JP200, JP201: LCSC C2337 -> (none)
- R400: LCSC C137954 -> (none)
- U400: LCSC C22445414 -> (none)
Changed lines of the file:
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@@
-			)
-		)
-		(property "LCSC" "C1525"
-			(at 46.99 40.6399 0)
-			(effects
-				(font
-					(size 1.27 1.27)
-				)
-				(hide yes)
 			)
 		)
@@
 			)
 		)
-		(property "LCSC" "C2337"
-			(at 111.76 64.7699 0)
-			(effects
-				(font
-					(size 1.27 1.27)
-				)
-				(hide yes)
-			)
-		)
 		(property "Sim.Device" ""
 			(at 109.22 66.04 0)
@@
 			)
 		)
-		(property "LCSC" "C2337"
-			(at 99.0601 49.53 0)
-			(effects
-				(font
-					(size 1.27 1.27)
-				)
-				(hide yes)
-			)
-		)
 		(property "Sim.Device" ""
 			(at 97.79 48.26 0)
@@
 			)
 		)
-		(property "LCSC" "C22445414"
-			(at 56.9595 52.07 0)
-			(effects
-				(font
-					(size 1.27 1.27)
-				)
-				(hide yes)
-			)
-		)
 		(property "Sim.Device" ""
 			(at 54.61 64.77 0)
@@
 			)
 		)
-		(property "LCSC" "C1525"
-			(at 26.67 74.9299 0)
-			(effects
-				(font
-					(size 1.27 1.27)
-				)
-				(hide yes)
-			)
-		)
 		(property "Sim.Device" ""
 			(at 22.86 76.2 0)
@@
 			)
 		)
-		(property "LCSC" "C2337"
-			(at 78.7401 49.53 0)
-			(effects
-				(font
-					(size 1.27 1.27)
-				)
-				(hide yes)
-			)
-		)
 		(property "Sim.Device" ""
 			(at 77.47 48.26 0)
@@
 			(effects
 				(font
-					(size 1.27 1.27)
-				)
-				(hide yes)
-			)
-		)
-		(property "LCSC" "C137954"
-			(at 85.852 56.896 0)
-			(effects
-				(font

Commit message: Document setup, update template, and use an ampersand when referring to APRL
Other:
- company: Aggie Propulsion and Rocketry Lab -> Aggie Propulsion & Rocketry Lab
Changed lines of the file:
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@@
 		(date "2025-10-15")
 		(rev "1A")
-		(company "Aggie Propulsion and Rocketry Lab")
+		(company "Aggie Propulsion & Rocketry Lab")
 		(comment 1 "Drawn by: Nolan Poe")
 		(comment 2 "Checked by: Daniel Fan")
