File: ali/v1/ThermoBoard/ethernet.kicad_sch (KiCad schematic)
At the start: 23 parts, among them J200 RJ45_Hanrun_HR911105A_Horizon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, U200 LAN8742A, Y200 25MHz

Commit message: Globally remove LCSC labels, update MPNs and IOCs, add +5V monitoring to DAQs, fix some footprints
Parts:
- C200, C206, C207: LCSC C602037 -> (none)
- C201, C203: LCSC C32949 -> (none)
- C202, C204, C205, C208: LCSC C1525 -> (none)
- J200: LCSC C12074 -> (none)
- R200, R202, R203: LCSC C60490 -> (none)
- R201: LCSC C138002 -> (none)
- R204, R206, R207, R208: LCSC C87044 -> (none)
- R205: LCSC C25852 -> (none)
- R209, R210: LCSC C105875 -> (none)
- Y200: LCSC C5765970 -> (none)
Changed lines of the file:
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@@
-			)
-		)
-		(property "LCSC" "C32949"
-			(at 45.72 144.7799 0)
-			(effects
-				(font
-					(size 1.27 1.27)
-				)
-				(hide yes)
 			)
 		)
@@
 			)
 		)
-		(property "LCSC" "C602037"
-			(at 41.91 52.0699 0)
-			(effects
-				(font
-					(size 1.27 1.27)
-				)
-				(hide yes)
-			)
-		)
 		(property "Sim.Device" ""
 			(at 38.1 53.34 0)
@@
 			)
 		)
-		(property "LCSC" "C602037"
-			(at 106.68 58.4199 0)
-			(effects
-				(font
-					(size 1.27 1.27)
-				)
-				(hide yes)
-			)
-		)
 		(property "Sim.Device" ""
 			(at 102.87 59.69 0)
@@
 			)
 		)
-		(property "LCSC" "C87044"
-			(at 134.62 77.4699 0)
-			(effects
-				(font
-					(size 1.27 1.27)
-				)
-				(hide yes)
-			)
-		)
 		(property "Sim.Device" ""
 			(at 132.08 78.74 0)
@@
 			)
 		)
-		(property "LCSC" "C12074"
-			(at 215.9 123.19 0)
-			(effects
-				(font
-					(size 1.27 1.27)
-				)
-				(hide yes)
-			)
-		)
 		(property "Sim.Device" ""
 			(at 214.63 137.16 0)
@@
 			)
 		)
-		(property "LCSC" "C138002"
-			(at 53.34 109.474 0)
-			(effects
-				(font
-					(size 1.27 1.27)
-				)
-				(hide yes)
-			)
-		)
 		(property "Sim.Device" ""
 			(at 58.42 110.49 90)
@@
 			)
 		)
-		(property "LCSC" "C1525"
-			(at 53.34 52.0699 0)
-			(effects
-				(font
-					(size 1.27 1.27)
-				)
-				(hide yes)
-			)
-		)
 		(property "Sim.Device" ""
 			(at 49.53 53.34 0)
@@
 			)
 		)
-		(property "LCSC" "C1525"
-			(at 76.2 52.0699 0)
-			(effects
-				(font
-					(size 1.27 1.27)
-				)
-				(hide yes)
-			)
-		)
 		(property "Sim.Device" ""
 			(at 72.39 53.34 0)
@@
 			)
 		)
-		(property "LCSC" "C60490"
-			(at 57.15 94.234 0)
-			(effects
-				(font
-					(size 1.27 1.27)
-				)
-				(hide yes)
-			)
-		)
 		(property "Sim.Device" ""
 			(at 62.23 95.25 90)
@@
 			)
 		)
-		(property "LCSC" "C87044"
-			(at 168.91 77.4699 0)
-			(effects
-				(font
-					(size 1.27 1.27)
-				)
-				(hide yes)
-			)
-		)
 		(property "Sim.Device" ""
 			(at 166.37 78.74 0)
@@
 			)
 		)
-		(property "LCSC" "C1525"
-			(at 187.96 147.3199 0)
-			(effects
-				(font
-					(size 1.27 1.27)
-				)
-				(hide yes)
-			)
-		)
 		(property "Sim.Device" ""
 			(at 184.15 148.59 0)
@@
 			)
 		)
-		(property "LCSC" "C602037"
-			(at 118.11 58.4199 0)
-			(effects
-				(font
-					(size 1.27 1.27)
-				)
-				(hide yes)
-			)
-		)
 		(property "Sim.Device" ""
 			(at 114.3 59.69 0)
@@
 			)
 		)
-		(property "LCSC" "C25852"
-			(at 135.89 105.4099 0)
-			(effects
-				(font
-					(size 1.27 1.27)
-				)
-				(hide yes)
-			)
-		)
 		(property "Sim.Device" ""
 			(at 133.35 106.68 0)
@@
 			)
 		)
-		(property "LCSC" "C5765970"
-			(at 61.214 129.032 0)
-			(effects
-				(font
-					(size 1.27 1.27)
-				)
-				(hide yes)
-			)
-		)
 		(property "Sim.Device" ""
 			(at 50.8 130.81 0)
@@
 			)
 		)
-		(property "LCSC" "C32949"
-			(at 60.96 144.7799 0)
-			(effects
-				(font
-					(size 1.27 1.27)
-				)
-				(hide yes)
-			)
-		)
 		(property "Sim.Device" ""
 			(at 57.15 146.05 0)
@@
 			)
 		)
-		(property "LCSC" "C87044"
-			(at 146.05 77.4699 0)
-			(effects
-				(font
-					(size 1.27 1.27)
-				)
-				(hide yes)
-			)
-		)
 		(property "Sim.Device" ""
 			(at 143.51 78.74 0)
@@
 			)
 		)
-		(property "LCSC" "C1525"
-			(at 64.77 52.0699 0)
-			(effects
-				(font
-					(size 1.27 1.27)
-				)
-				(hide yes)
-			)
-		)
 		(property "Sim.Device" ""
 			(at 60.96 53.34 0)
@@
 			)
 		)
-		(property "LCSC" "C105875"
-			(at 259.08 137.1599 0)
-			(effects
-				(font
-					(size 1.27 1.27)
-				)
-				(hide yes)
-			)
-		)
 		(property "Sim.Device" ""
 			(at 256.54 138.43 0)
@@
 			)
 		)
-		(property "LCSC" "C60490"
-			(at 115.57 113.0299 0)
-			(effects
-				(font
-					(size 1.27 1.27)
-				)
-				(hide yes)
-			)
-		)
 		(property "Sim.Device" ""
 			(at 113.03 114.3 0)
@@
 			)
 		)
-		(property "LCSC" "C60490"
-			(at 50.8 74.9299 0)
-			(effects
-				(font
-					(size 1.27 1.27)
-				)
-				(hide yes)
-			)
-		)
 		(property "Sim.Device" ""
 			(at 48.26 76.2 0)
@@
 			)
 		)
-		(property "LCSC" "C105875"
-			(at 250.19 147.3199 0)
-			(effects
-				(font
-					(size 1.27 1.27)
-				)
-				(hide yes)
-			)
-		)
 		(property "Sim.Device" ""
 			(at 247.65 148.59 0)
@@
 			(effects
 				(font
-					(size 1.27 1.27)
-				)
-				(hide yes)
-			)
-		)
-		(property "LCSC" "C87044"
-			(at 157.48 77.4699 0)
-			(effects
-				(font

Commit message: Document setup, update template, and use an ampersand when referring to APRL
Other:
- company: Aggie Propulsion and Rocketry Lab -> Aggie Propulsion & Rocketry Lab
Changed lines of the file:
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@@
 		(date "2025-10-15")
 		(rev "1A")
-		(company "Aggie Propulsion and Rocketry Lab")
+		(company "Aggie Propulsion & Rocketry Lab")
 		(comment 1 "Drawn by: Nolan Poe")
 		(comment 2 "Checked by: Daniel Fan")
