File: ali/v1/ThermoBoard/microcontroller.kicad_sch (KiCad schematic)
At the start: 52 parts, among them J100 Conn_01x05_Pin, J101 Screw_Terminal_01x02, J102 USB_C_Receptacle_USB2.0_16P, Q100 Si2371EDS, SW100 SKRPANE010, U100 STM32H563RITx, U101 AP2112K-3.3, U102 USBLC6-2SC6, Y100 16MHz

Commit message: Globally remove LCSC labels, update MPNs and IOCs, add +5V monitoring to DAQs, fix some footprints
Parts:
- C100, C103, C106, C108, C114, C115, C116: LCSC C602037 -> (none)
- C101, C102, C105, C110, C112, C113, C117: LCSC C1525 -> (none)
- C104, C107: LCSC C32949 -> (none)
- C109, C111: LCSC C170151 -> (none)
- C118, C119: LCSC C15849 -> (none)
- D100, D101, D102, D103, D105: LCSC C965793 -> (none)
- D104: LCSC C39057 -> (none)
- F100: LCSC C19193036 -> (none)
- F101: LCSC C22435898 -> (none)
- J100, JP100: LCSC C2337 -> (none)
- J101: LCSC C3029316 -> (none)
- J102: LCSC C165948 -> (none)
- Q100: LCSC C467897 -> (none)
- R100, R101, R102, R103, R107: LCSC C105875 -> (none)
- R104: LCSC C60490 -> (none)
- R105, R106: LCSC C105873 -> (none)
- SW100: LCSC C2909692 -> (none)
- U100: LCSC C20619634 -> (none)
- U101: LCSC C51118 -> (none)
- U102: LCSC C7519 -> (none)
- Y100: LCSC C2901668 -> (none)

Commit message: Document setup, update template, and use an ampersand when referring to APRL
Other:
- company: Aggie Propulsion and Rocketry Lab -> Aggie Propulsion & Rocketry Lab
Changed lines of the file:
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@@
 		(date "2025-10-15")
 		(rev "1A")
-		(company "Aggie Propulsion and Rocketry Lab")
+		(company "Aggie Propulsion & Rocketry Lab")
 		(comment 1 "Drawn by: Nolan Poe")
 		(comment 2 "Checked by: Daniel Fan")
