File: ali/v1/ThermoBoard/thermocouples.kicad_sch (KiCad schematic)
At the start: 52 parts, among them J300 PCC-SMP-K-5, J301 PCC-SMP-K-5, J302 PCC-SMP-K-5, J303 PCC-SMP-K-5, U300 MAX31856, U301 MAX31856, U302 MAX31856, U303 MAX31856

Commit message: Globally remove LCSC labels, update MPNs and IOCs, add +5V monitoring to DAQs, fix some footprints
Parts:
- C300, C302, C303, C305, C310, C312, C313, C315: LCSC C15195 -> (none)
- C301, C304, C306, C307, C308, C309, C311, C314, C316, C317, C318, C319: LCSC C1525 -> (none)
- D300, D301, D302, D303: LCSC C21260817 -> (none)
- R300, R301, R304, R305: LCSC C60490 -> (none)
- R302, R303, R306, R307: LCSC C105875 -> (none)
- U300, U301, U302, U303: LCSC C2653162 -> (none)

Commit message: Document setup, update template, and use an ampersand when referring to APRL
Other:
- company: Aggie Propulsion and Rocketry Lab -> Aggie Propulsion & Rocketry Lab
Changed lines of the file:
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@@
 		(date "2025-10-15")
 		(rev "1A")
-		(company "Aggie Propulsion and Rocketry Lab")
+		(company "Aggie Propulsion & Rocketry Lab")
 		(comment 1 "Drawn by: Nolan Poe")
 		(comment 2 "Checked by: Daniel Fan")
