File: kicadlibs/templates/ali_v2/microcontroller.kicad_sch (KiCad schematic)
At the start: 39 parts, among them J1 Conn_02x01, J2 Conn_01x05, J3 USB_C_Receptacle_USB2.0_16P, J6 Screw_Terminal_01x02, SW1 SKRPANE010, U1 STM32H563RIV6, U2 AP2112K-3.3, Y1 25 MHz

Commit message: Begin prep for second board review
Parts:
- R1, R2: value 4.7k -> 5.1k; MPN RC0603FR-074K7L -> RC0603FR-075K1L
Changed lines of the file:
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@@
 	(paper "USLetter")
 	(title_block
-		(date "2026-09-11")
+		(date "2026-10-10")
 	)
